File: tracker/hardware/hub_board_diy/hub_board_diy.kicad_sch (KiCad schematic)
At the start: 12 parts, among them U1 ESP32-C3_Mini_V1, U2L LoRa2021_Left, U2R LoRa2021_Right, U3 BMP280

Commit message: feat: extend DIY v0.1 schematic with GPS, power chain, learnings notes
Added: GPS connector (MAX-M10S), BAT54 diode, TPS7A02 LDO, supercap pads,
SB3 power select, solar input, ADC voltage divider, debug header, C5-C7.
Added text notes: SPI 20MHz layout rules, strapping pin warnings,
RadioLib config requirements, power chain description.
Parts:
- added C5, C7: 100nF, Capacitor_SMD:C_0805_2012Metric, symbol Device:C
- added C6: 10uF, Capacitor_SMD:C_0805_2012Metric, symbol Device:C
- added D1: BAT54, Diode_SMD:D_SOT-23, symbol Device:D_Schottky
- added J1: Debug, Connector_PinHeader_2.54mm:PinHeader_2x03_P2.54mm_Vertical, symbol Connector_Generic:Conn_02x03_Odd_Even
- added J2: Solar_In, Connector_PinHeader_2.54mm:PinHeader_1x02_P2.54mm_Vertical, symbol Connector_Generic:Conn_01x02
- added R1, R2: 1M, Resistor_SMD:R_0805_2012Metric, symbol Device:R
- added SB3: PWR_SEL, Jumper:SolderJumper-3_P1.3mm_Bridged12_Pad1.0x1.5mm, symbol Jumper:SolderJumper_3_Bridged12
- added SC1: 1.0F 5.5V, Capacitor_THT:CP_Radial_D8.0mm_P3.50mm, symbol Device:C_Polarized
- added U4: MAX-M10S, Connector_PinHeader_2.54mm:PinHeader_1x04_P2.54mm_Vertical, symbol Connector_Generic:Conn_01x04_Pin
- added U5: TPS7A0233DBVR, Package_TO_SOT_SMD:SOT-23-3, symbol Regulator_Linear:AP2112_SA23_SOT23_3
Other:
- note added: "POWER CHAIN: Solar→BAT54→1.0F supercap→TPS7A02→3.3V. SB3 selects USB vs solar power."
- note added: "RADIOLIB: Set radio.irqDioNum=9 before begin(). Pass tcxoVoltage=0 (LR2021 uses XTAL, not TCXO)."
- note added: "SPI LAYOUT: 20MHz continuous SCK proven. Traces <30mm, length-matched ~5mm. Ground plane under SPI bus."
- note added: "STRAPPING PINS: GPIO8=HIGH at boot (download mode if pulled low). GPIO9=LOW at boot (download mode). Do NOT use for I2C with pullups on flight board — use GPIO20/GPIO21 instead."
Changed lines of the file:
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@@
     (uuid "text-0001")
   )
+  ;; ========== GPS CONNECTOR (U4) ==========
+  (symbol (lib_id "Connector_Generic:Conn_01x04_Pin") (at 63.5 116.84 0) (unit 1)
+    (in_bom yes) (on_board yes)
+    (property "Reference" "U4" (at 64.77 109.22 0) (effects (font (size 1.27 1.27))))
+    (property "Value" "MAX-M10S" (at 64.77 111.76 0) (effects (font (size 1.27 1.27))))
+    (property "Footprint" "Connector_PinHeader_2.54mm:PinHeader_1x04_P2.54mm_Vertical" (at 63.5 116.84 0) (effects (font (size 1.27 1.27)) hide))
+    (property "Datasheet" "~" (at 63.5 116.84 0) (effects (font (size 1.27 1.27)) hide))
+    (pin "1")
+    (pin "2")
+    (pin "3")
+    (pin "4")
+  )
+  ;; ========== BAT54 SCHOTTKY DIODE (D1) ==========
+  (symbol (lib_id "Device:D_Schottky") (at 30.48 93.98 0) (unit 1)
+    (in_bom yes) (on_board yes)
+    (property "Reference" "D1" (at 30.48 88.9 0) (effects (font (size 1.27 1.27))))
+    (property "Value" "BAT54" (at 30.48 91.44 0) (effects (font (size 1.27 1.27))))
+    (property "Footprint" "Diode_SMD:D_SOT-23" (at 30.48 93.98 0) (effects (font (size 1.27 1.27)) hide))
+    (property "Datasheet" "~" (at 30.48 93.98 0) (effects (font (size 1.27 1.27)) hide))
+    (pin "1")
+    (pin "2")
+  )
+  ;; ========== TPS7A02 LDO (U5) ==========
+  (symbol (lib_id "Regulator_Linear:AP2112_SA23_SOT23_3") (at 30.48 83.82 0) (unit 1)
+    (in_bom yes) (on_board yes)
+    (property "Reference" "U5" (at 30.48 76.2 0) (effects (font (size 1.27 1.27))))
+    (property "Value" "TPS7A0233DBVR" (at 30.48 78.74 0) (effects (font (size 1.27 1.27))))
+    (property "Footprint" "Package_TO_SOT_SMD:SOT-23-3" (at 30.48 83.82 0) (effects (font (size 1.27 1.27)) hide))
+    (property "Datasheet" "~" (at 30.48 83.82 0) (effects (font (size 1.27 1.27)) hide))
+    (pin "1")
+    (pin "2")
+    (pin "3")
+  )
+  ;; ========== SUPERCAP PADS (SC1) ==========
+  (symbol (lib_id "Device:C_Polarized") (at 20.32 93.98 0) (unit 1)
+    (in_bom yes) (on_board yes)
+    (property "Reference" "SC1" (at 17.78 88.9 0) (effects (font (size 1.27 1.27)) (justify right)))
+    (property "Value" "1.0F 5.5V" (at 17.78 91.44 0) (effects (font (size 1.27 1.27)) (justify right)))
+    (property "Footprint" "Capacitor_THT:CP_Radial_D8.0mm_P3.50mm" (at 20.32 93.98 0) (effects (font (size 1.27 1.27)) hide))
+    (property "Datasheet" "~" (at 20.32 93.98 0) (effects (font (size 1.27 1.27)) hide))
+    (pin "1")
+    (pin "2")
+  )
+  ;; ========== POWER SELECT JUMPER (SB3) ==========
+  (symbol (lib_id "Jumper:SolderJumper_3_Bridged12") (at 30.48 73.66 0) (unit 1)
+    (in_bom no) (on_board yes)
+    (property "Reference" "SB3" (at 30.48 68.58 0) (effects (font (size 1.27 1.27))))
+    (property "Value" "PWR_SEL" (at 30.48 71.12 0) (effects (font (size 1.27 1.27))))
+    (property "Footprint" "Jumper:SolderJumper-3_P1.3mm_Bridged12_Pad1.0x1.5mm" (at 30.48 73.66 0) (effects (font (size 1.27 1.27)) hide))
+    (pin "1")
+    (pin "2")
+    (pin "3")
+  )
+  ;; ========== SOLAR INPUT PADS (J2) ==========
+  (symbol (lib_id "Connector_Generic:Conn_01x02") (at 15.24 93.98 0) (unit 1)
+    (in_bom yes) (on_board yes)
+    (property "Reference" "J2" (at 15.24 88.9 0) (effects (font (size 1.27 1.27))))
+    (property "Value" "Solar_In" (at 15.24 91.44 0) (effects (font (size 1.27 1.27))))
+    (property "Footprint" "Connector_PinHeader_2.54mm:PinHeader_1x02_P2.54mm_Vertical" (at 15.24 93.98 0) (effects (font (size 1.27 1.27)) hide))
+    (property "Datasheet" "~" (at 15.24 93.98 0) (effects (font (size 1.27 1.27)) hide))
+    (pin "1")
+    (pin "2")
+  )
+  ;; ========== ADC VOLTAGE DIVIDER R1 ==========
+  (symbol (lib_id "Device:R") (at 40.64 93.98 0) (unit 1)
+    (in_bom yes) (on_board yes)
+    (property "Reference" "R1" (at 43.18 91.44 0) (effects (font (size 1.27 1.27)) (justify left)))
+    (property "Value" "1M" (at 43.18 96.52 0) (effects (font (size 1.27 1.27)) (justify left)))
+    (property "Footprint" "Resistor_SMD:R_0805_2012Metric" (at 40.64 93.98 0) (effects (font (size 1.27 1.27)) hide))
+    (property "Datasheet" "~" (at 40.64 93.98 0) (effects (font (size 1.27 1.27)) hide))
+    (pin "1")
+    (pin "2")
+  )
+  ;; ========== ADC VOLTAGE DIVIDER R2 ==========
+  (symbol (lib_id "Device:R") (at 40.64 101.6 0) (unit 1)
+    (in_bom yes) (on_board yes)
+    (property "Reference" "R2" (at 43.18 99.06 0) (effects (font (size 1.27 1.27)) (justify left)))
+    (property "Value" "1M" (at 43.18 104.14 0) (effects (font (size 1.27 1.27)) (justify left)))
+    (property "Footprint" "Resistor_SMD:R_0805_2012Metric" (at 40.64 101.6 0) (effects (font (size 1.27 1.27)) hide))
+    (property "Datasheet" "~" (at 40.64 101.6 0) (effects (font (size 1.27 1.27)) hide))
+    (pin "1")
+    (pin "2")
+  )
+  ;; ========== DEBUG HEADER (J1) ==========
+  (symbol (lib_id "Connector_Generic:Conn_02x03_Odd_Even") (at 170.18 73.66 0) (unit 1)
+    (in_bom yes) (on_board yes)
+    (property "Reference" "J1" (at 170.18 66.04 0) (effects (font (size 1.27 1.27))))
+    (property "Value" "Debug" (at 170.18 68.58 0) (effects (font (size 1.27 1.27))))
+    (property "Footprint" "Connector_PinHeader_2.54mm:PinHeader_2x03_P2.54mm_Vertical" (at 170.18 73.66 0) (effects (font (size 1.27 1.27)) hide))
+    (property "Datasheet" "~" (at 170.18 73.66 0) (effects (font (size 1.27 1.27)) hide))
+    (pin "1")
+    (pin "2")
+    (pin "3")
+    (pin "4")
+    (pin "5")
+    (pin "6")
+  )
+  ;; ========== C5: GPS DECOUPLE 100nF ==========
+  (symbol (lib_id "Device:C") (at 73.66 93.98 0) (unit 1)
+    (in_bom yes) (on_board yes)
+    (property "Reference" "C5" (at 76.2 91.44 0) (effects (font (size 1.27 1.27)) (justify left)))
+    (property "Value" "100nF" (at 76.2 96.52 0) (effects (font (size 1.27 1.27)) (justify left)))
+    (property "Footprint" "Capacitor_SMD:C_0805_2012Metric" (at 73.66 93.98 0) (effects (font (size 1.27 1.27)) hide))
+    (property "Datasheet" "~" (at 73.66 93.98 0) (effects (font (size 1.27 1.27)) hide))
+    (pin "1")
+    (pin "2")
+  )
+  ;; ========== C6: GPS DECOUPLE 10uF ==========
+  (symbol (lib_id "Device:C") (at 83.82 93.98 0) (unit 1)
+    (in_bom yes) (on_board yes)
+    (property "Reference" "C6" (at 86.36 91.44 0) (effects (font (size 1.27 1.27)) (justify left)))
+    (property "Value" "10uF" (at 86.36 96.52 0) (effects (font (size 1.27 1.27)) (justify left)))
+    (property "Footprint" "Capacitor_SMD:C_0805_2012Metric" (at 83.82 93.98 0) (effects (font (size 1.27 1.27)) hide))
+    (property "Datasheet" "~" (at 83.82 93.98 0) (effects (font (size 1.27 1.27)) hide))
+    (pin "1")
+    (pin "2")
+  )
+  ;; ========== C7: LDO OUTPUT 100nF ==========
+  (symbol (lib_id "Device:C") (at 40.64 83.82 0) (unit 1)
+    (in_bom yes) (on_board yes)
+    (property "Reference" "C7" (at 43.18 81.28 0) (effects (font (size 1.27 1.27)) (justify left)))
+    (property "Value" "100nF" (at 43.18 86.36 0) (effects (font (size 1.27 1.27)) (justify left)))
+    (property "Footprint" "Capacitor_SMD:C_0805_2012Metric" (at 40.64 83.82 0) (effects (font (size 1.27 1.27)) hide))
+    (property "Datasheet" "~" (at 40.64 83.82 0) (effects (font (size 1.27 1.27)) hide))
+    (pin "1")
+    (pin "2")
+  )
+  ;; ========== NEW LABELS ==========
+  (label "UART1_TX" (at 48.26 111.76 0) (fields_autoplaced)
+    (effects (font (size 1.27 1.27)) (justify left bottom))
+    (uuid "label-0012")
+  )
+  (label "UART1_RX" (at 48.26 114.3 0) (fields_autoplaced)
+    (effects (font (size 1.27 1.27)) (justify left bottom))
+    (uuid "label-0013")
+  )
+  (label "ADC_VCAP" (at 48.26 99.06 0) (fields_autoplaced)
+    (effects (font (size 1.27 1.27)) (justify left bottom))
+    (uuid "label-0014")
+  )
+  ;; ========== LEARNINGS TEXT NOTES ==========
+  (text "SPI LAYOUT: 20MHz continuous SCK proven. Traces <30mm, length-matched ~5mm. Ground plane under SPI bus."
+    (at 170.18 20.32 0)
+    (effects (font (size 1.27 1.27)) (justify left))
+    (uuid "text-0002")
+  )
+  (text "STRAPPING PINS: GPIO8=HIGH at boot (download mode if pulled low). GPIO9=LOW at boot (download mode). Do NOT use for I2C with pullups on flight board — use GPIO20/GPIO21 instead."
+    (at 170.18 30.48 0)
+    (effects (font (size 1.27 1.27)) (justify left))
+    (uuid "text-0003")
+  )
+  (text "RADIOLIB: Set radio.irqDioNum=9 before begin(). Pass tcxoVoltage=0 (LR2021 uses XTAL, not TCXO)."
+    (at 170.18 40.64 0)
+    (effects (font (size 1.27 1.27)) (justify left))
+    (uuid "text-0004")
+  )
+  (text "POWER CHAIN: Solar→BAT54→1.0F supercap→TPS7A02→3.3V. SB3 selects USB vs solar power."
+    (at 170.18 50.8 0)
+    (effects (font (size 1.27 1.27)) (justify left))
+    (uuid "text-0005")
+  )
 )
