File: tracker/hardware/output/v1_freerouted_final.kicad_pcb (KiCad board)
At the start: 2 copper layers, 50 x 40 mm, 30 parts, among them U1 RP2040-Zero, U2 LoRa2021, U3 MAX-M10S, U4 MS5611, U5 TPS7A02

Commit message: wip: Freerouting DSN pipeline — 241 tracks imported, GND zone fill, coordinate investigation
- Persisted /tmp/routed_output.dsn and /tmp/clean_export.dsn to repo
- import_freerouting_final.py: imports Freerouting tracks, fills GND zone
- route_power_nets.py: power net routing attempt (made violations worse)
- PCB-REMAINING-ISSUES-ANALYSIS.md: root cause analysis
- KNOWN ISSUE: DSN Y-axis negation — tracks land at negative Y, pads at positive Y
- Y flip correct but creates overlaps (512 violations vs 269 without flip)
- GND copper pour exists on F.Cu but blocked by misaligned tracks
Routing:
- net I2C_SDA: track 1402.0 -> 0.00 mm
- net 3V3: track 0.00 -> 1402.0 mm
