File: tracker/hardware/output/v2_adc_clean2.kicad_pcb (KiCad board)
At the start: 2 copper layers, 50 x 40 mm, 17 parts, among them U1 ESP32-C3, U2 LR2021F33, U3 MAX-M10S, U4 TPS7A02

Commit message: persist: remaining kimi-k3 scripts + SES files + DRC results
Routing:
- net 3V3: track 10.2 -> 60.4 mm
- net RF_SUB_868: track 0.00 -> 36.0 mm
- net VDIV_MID: track 45.1 -> 20.6 mm, vias 2 -> 1
- net VCAP: track 0.77 -> 22.7 mm
- net LR2021_DIO9: track 0.00 -> 21.5 mm
- net GND: track 83.1 -> 103.9 mm
- net RF_2G4_2400: track 0.00 -> 16.2 mm
- net STATUS_LED: track 0.00 -> 10.5 mm
- net LR2021_BUSY: track 0.00 -> 9.93 mm
- net SPI_NSS: track 0.00 -> 9.12 mm
- net SPI_MISO: track 0.00 -> 6.21 mm
- net SPI_SCK: track 0.00 -> 4.52 mm
Changed lines of the file:
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@@
+	)
+	(segment
+		(start 8.9 18.8)
+		(end 9.5 22)
+		(width 0.4)
+		(layer "F.Cu")
+		(net 1)
+	)
+	(segment
+		(start 8.9 18.8)
+		(end 10.9 12)
+		(width 0.4)
+		(layer "F.Cu")
+		(net 1)
 	)
 	(segment
@@
 	)
 	(segment
+		(start 15.5 8.199999)
+		(end 40 25)
+		(width 0.4)
+		(layer "F.Cu")
+		(net 1)
+	)
+	(segment
 		(start 1.6249 29.6253)
 		(end 1.9996 30)
@@
 	)
 	(segment
+		(start 1.6 28.4)
+		(end 9.5 22)
+		(width 0.4)
+		(layer "F.Cu")
+		(net 1)
+	)
+	(segment
 		(start 1.5998 29.6002)
 		(end 1.6249 29.6253)
@@
 	)
 	(segment
+		(start 10.5 20)
+		(end 10.5 22)
+		(width 0.25)
+		(layer "F.Cu")
+		(net 2)
+	)
+	(segment
 		(start 32.5 14)
 		(end 32.5 24)
@@
 	)
 	(segment
+		(start 10.5 22)
+		(end 12.1 26)
+		(width 0.25)
+		(layer "F.Cu")
+		(net 2)
+	)
+	(segment
+		(start 10.1 14)
+		(end 8 17.2)
+		(width 0.25)
+		(layer "F.Cu")
+		(net 2)
+	)
+	(segment
 		(start 10 13.9)
 		(end 10.1 14)
@@
 		(end 24.1999 7.6999)
 		(width 0.7998)
+		(layer "F.Cu")
+		(net 2)
+	)
+	(segment
+		(start 5 31.4)
+		(end 3.3 28)
+		(width 0.25)
 		(layer "F.Cu")
 		(net 2)
@@
 		(end 10.1 26)
 		(width 2)
+		(layer "F.Cu")
+		(net 2)
+	)
+	(segment
+		(start 15.5 9.8)
+		(end 10 13.9)
+		(width 0.25)
 		(layer "F.Cu")
 		(net 2)
@@
 	)
 	(segment
+		(start 10.1 20)
+		(end 10.5 15.5)
+		(width 0.25)
+		(layer "F.Cu")
+		(net 3)
+	)
+	(segment
 		(start 12.2632 17.2389)
 		(end 11.9019 17.6002)
@@
 		(layer "F.Cu")
 		(net 4)
+	)
+	(segment
+		(start 10.1 16)
+		(end 11 13)
+		(width 0.25)
+		(layer "F.Cu")
+		(net 5)
+	)
+	(segment
+		(start 11 13)
+		(end 8.5 11.2)
+		(width 0.25)
+		(layer "F.Cu")
+		(net 5)
+	)
+	(segment
+		(start 10.1 22)
+		(end 16.5 15.5)
+		(width 0.25)
+		(layer "F.Cu")
+		(net 6)
+	)
+	(segment
+		(start 8.5 14.2)
+		(end 10.1 24)
+		(width 0.25)
+		(layer "F.Cu")
+		(net 7)
 	)
 	(segment
@@
 	)
 	(segment
+		(start 8.5 15.8)
+		(end 29.9 18)
+		(width 0.25)
+		(layer "F.Cu")
+		(net 9)
+	)
+	(segment
 		(start 4.517 9.75)
 		(end 6.7981 9.75)
@@
 	)
 	(segment
+		(start 15 15.5)
+		(end 19.5 6)
+		(width 0.25)
+		(layer "F.Cu")
+		(net 11)
+	)
+	(segment
 		(start 20.5 6)
 		(end 21.5 6)
@@
 		(end 7 17.3)
 		(width 0.3998)
+		(layer "F.Cu")
+		(net 13)
+	)
+	(segment
+		(start 9.5 20)
+		(end 8.9 17.2)
+		(width 0.4)
+		(layer "F.Cu")
+		(net 13)
+	)
+	(segment
+		(start 7.5 37)
+		(end 9.5 20)
+		(width 0.4)
+		(layer "F.Cu")
+		(net 13)
+	)
+	(segment
+		(start 8.9 17.2)
+		(end 7 17.3)
+		(width 0.4)
 		(layer "F.Cu")
 		(net 13)
@@
 	)
 	(segment
+		(start 10.1 28)
+		(end 46 25)
+		(width 0.76)
+		(layer "F.Cu")
+		(net 16)
+	)
+	(segment
+		(start 29.9 28)
+		(end 46 30)
+		(width 0.76)
+		(layer "F.Cu")
+		(net 17)
+	)
+	(segment
 		(start 10.2019 8.2498)
 		(end 8.5002 8.2498)
@@
 		(end 2.8356 33.5854)
 		(width 2)
+		(layer "F.Cu")
+		(net 18)
+	)
+	(segment
+		(start 1.9 32.6)
+		(end 3.5 30)
+		(width 0.25)
 		(layer "F.Cu")
 		(net 18)
@@
 		(net 18)
 	)
-	(via
-		(at 10.6521 8.2498)
-		(size 0.6)
-		(drill 0.3)
-		(layers "F.Cu" "B.Cu")
-		(net 18)
-	)
-	(segment
-		(start 10.6521 8.2498)
-		(end 16.0072 13.6049)
-		(width 2)
-		(layer "B.Cu")
-		(net 18)
-	)
-	(segment
-		(start 16.0072 13.6049)
-		(end 16.0072 33.5854)
-		(width 2)
-		(layer "B.Cu")
-		(net 18)
-	)

Commit message: feat: V2-ADC v3 board — kimi-k3 FreeRouting output, 0 violations, 22 unconnected
Best board yet: 0 shorts, 0 violations, 106 tracks, 12 vias.
22 unconnected pairs remain — board is saturated, needs manual KiCad GUI finish.

Unconnected pairs by distance:
- 7 pairs <5mm (VCAP, VDIV_MID, SPI_MISO, 4xGND)
- 5 pairs 5-10mm (3V3, SPI_MOSI, SPI_MISO, 2xGND)
- 10 pairs >10mm (SPI_SCK, SPI_NSS, LR2021_BUSY, LR2021_RST, GPS_RX, STATUS_LED, FEM_TX, RF, 3V3, GND)

Estimated manual finish: 45-75 min in KiCad GUI (interactive rip-up-and-retry).
Headless auto-routing cannot converge — board is too dense for naive track insertion.
Routing:
- net GND: track 103.9 -> 127.8 mm
- net VDIV_MID: track 20.6 -> 7.00 mm, vias 1 -> 0
Changed lines of the file:
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@@
+	)
+	(segment
+		(start 41.5 25)
+		(end 29.9 24)
+		(width 0.25)
+		(layer "F.Cu")
+		(net 2)
 	)
 	(segment
@@
 		(end 12.0617 28.9462)
 		(width 2)
+		(layer "F.Cu")
+		(net 2)
+	)
+	(segment
+		(start 10 31.1)
+		(end 12.5 37)
+		(width 0.25)
 		(layer "F.Cu")
 		(net 2)
@@
 		(end 44.5 30)
 		(width 2)
+		(layer "B.Cu")
+		(net 2)
+	)
+	(segment
+		(start 44.5 30)
+		(end 41.5 25)
+		(width 0.25)
 		(layer "B.Cu")
 		(net 2)
@@
 		(net 18)
 	)
-	(segment
-		(start 10.6521 8.2498)
-		(end 10.2019 8.2498)
-		(width 2)
-		(layer "F.Cu")
-		(net 18)
-	)
-	(segment
-		(start 2.8356 33.5854)
-		(end 16.0072 33.5854)
-		(width 2)
-		(layer "F.Cu")
-		(net 18)
-	)
-	(segment
-		(start 8.5002 8.2498)
-		(end 8.5 8.25)
-		(width 0.5998)
-		(layer "F.Cu")
-		(net 18)
-	)
-	(via
-		(at 16.0072 33.5854)
-		(size 0.6)
-		(drill 0.3)
-		(layers "F.Cu" "B.Cu")
-		(net 18)
-	)
