File: tracker/hardware/output/v2_adc_v3.kicad_pcb (KiCad board)
At the start: 2 copper layers, 50 x 40 mm, 17 parts, among them U1 ESP32-C3, U2 LR2021F33, U3 MAX-M10S, U4 TPS7A02

Commit message: feat: V2-ADC v3 board — kimi-k3 FreeRouting output, 0 violations, 22 unconnected
Best board yet: 0 shorts, 0 violations, 106 tracks, 12 vias.
22 unconnected pairs remain — board is saturated, needs manual KiCad GUI finish.

Unconnected pairs by distance:
- 7 pairs <5mm (VCAP, VDIV_MID, SPI_MISO, 4xGND)
- 5 pairs 5-10mm (3V3, SPI_MOSI, SPI_MISO, 2xGND)
- 10 pairs >10mm (SPI_SCK, SPI_NSS, LR2021_BUSY, LR2021_RST, GPS_RX, STATUS_LED, FEM_TX, RF, 3V3, GND)

Estimated manual finish: 45-75 min in KiCad GUI (interactive rip-up-and-retry).
Headless auto-routing cannot converge — board is too dense for naive track insertion.
Routing:
- net GND: track 115.1 -> 147.2 mm
- net VDIV_MID: track 28.2 -> 2.24 mm, vias 2 -> 0
- net RF_SUB_868: track 54.7 -> 36.3 mm, vias 2 -> 1
- net 3V3: track 36.6 -> 45.6 mm
- net SPI_MOSI: track 0.00 -> 8.12 mm
- net SPI_MISO: track 0.00 -> 3.08 mm
- net VCAP: track 22.0 -> 23.9 mm
Changed lines of the file:
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@@
+	)
+	(segment
+		(start 15.5 8.199999)
+		(end 17.1 17)
+		(width 0.4)
+		(layer "F.Cu")
+		(net 1)
 	)
 	(segment
@@
 	)
 	(segment
+		(start 10 13)
+		(end 8 17.2)
+		(width 0.25)
+		(layer "F.Cu")
+		(net 2)
+	)
+	(segment
 		(start 6.2079 34.5993)
 		(end 6.2079 34.9642)
@@
 	)
 	(segment
+		(start 10.5 20)
+		(end 15.1 19)
+		(width 0.25)
+		(layer "F.Cu")
+		(net 2)
+	)
+	(segment
 		(start 4.1792 32.5706)
 		(end 6.2079 34.5993)
@@
 		(net 2)
 	)
+	(segment
+		(start 10.5 20)
+		(end 8 17.2)
+		(width 0.25)
+		(layer "F.Cu")
+		(net 2)
+	)
 	(via
 		(at 21.9345 7.966)
@@
 	)
 	(segment
+		(start 3.3 28)
+		(end 3.5 32)
+		(width 0.25)
+		(layer "B.Cu")
+		(net 2)
+	)
+	(segment
+		(start 37.5 31)
+		(end 44.5 30)
+		(width 0.25)
+		(layer "B.Cu")
+		(net 2)
+	)
+	(segment
+		(start 17.2 9.8)
+		(end 10 13)
+		(width 0.25)
+		(layer "B.Cu")
+		(net 2)
+	)
+	(segment
 		(start 21.9345 7.966)
 		(end 24.966 7.966)
@@
 	)
 	(segment
+		(start 12 15.5)
+		(end 15.1 23)
+		(width 0.25)
+		(layer "F.Cu")
+		(net 4)
+	)
+	(segment
+		(start 11 13)
+		(end 8.5 11.2)
+		(width 0.25)
+		(layer "F.Cu")
+		(net 5)
+	)
+	(segment
 		(start 8.2626 15.5126)
 		(end 7.4611 15.5126)
@@
 		(end 7.2002 18.2002)
 		(width 0.5998)
+		(layer "F.Cu")
+		(net 13)
+	)
+	(segment
+		(start 8.9 17.2)
+		(end 7 17.3)
+		(width 0.4)
 		(layer "F.Cu")
 		(net 13)
@@
 		(net 16)
 	)
-	(via
-		(at 27.6007 14.7935)
-		(size 0.76)
-		(drill 0.3)
-		(layers "F.Cu" "B.Cu")
-		(net 16)
-	)
-	(segment
-		(start 27.6007 33.2019)
-		(end 27.6007 14.7935)
-		(width 0.76)
-		(layer "B.Cu")
-		(net 16)
-	)
-	(segment
-		(start 5.3345 30)
-		(end 6.4432 28.8913)
-		(width 2)
+	(segment
+		(start 3.5 30)
+		(end 2.5 32)
+		(width 0.25)
 		(layer "F.Cu")
 		(net 18)
 	)
-	(segment
-		(start 6.4432 26.4666)
-		(end 4.9831 25.0065)
-		(width 2)
-		(layer "F.Cu")
-		(net 18)
-	)
-	(segment
-		(start 4.0019 30)
-		(end 3.5 30)
-		(width 0.4998)
-		(layer "F.Cu")
-		(net 18)
-	)
-	(segment
-		(start 6.4432 28.8913)
-		(end 6.4432 26.4666)
-		(width 2)
-		(layer "F.Cu")
-		(net 18)
-	)
-	(segment
-		(start 4.0019 30)
-		(end 5.3345 30)
-		(width 2)
-		(layer "F.Cu")
-		(net 18)
-	)
-	(segment
-		(start 8.5 8.25)
-		(end 4.9831 8.25)
-		(width 0.5998)
-		(layer "F.Cu")
-		(net 18)
-	)
-	(via
-		(at 4.9831 25.0065)
-		(size 0.6)
-		(drill 0.3)
-		(layers "F.Cu" "B.Cu")
-		(net 18)
-	)
-	(via
-		(at 4.9831 8.25)
-		(size 0.6)
-		(drill 0.3)
-		(layers "F.Cu" "B.Cu")
-		(net 18)
-	)
-	(segment
-		(start 4.9831 25.0065)
-		(end 4.9831 8.25)
-		(width 2)
-		(layer "B.Cu")
-		(net 18)
-	)
