File: tracker/hardware/output/v2_adc_fixed.kicad_pcb (KiCad board)
At the start: 2 copper layers, 50 x 40 mm, 17 parts, among them U1 ESP32-C3, U2 LR2021F33, U3 MAX-M10S, U4 TPS7A02

Commit message: feat: 2-LAYER V2-ADC board — BEST RESULT: 0v/16uc/0s + gerbers exported
Best 2-layer board: v2_adc_fixed2.kicad_pcb
- 0 violations, 0 shorts, 16 unconnected
- Gerbers exported: output/v2_adc_2layer_gerbers.zip

16 unconnected breakdown:
- CRITICAL: 2x3V3, 4xGND, SPI_SCK, LR2021_BUSY, LR2021_DIO9, VCAP, SOLAR_IN (11 critical)
- NON-CRITICAL: STATUS_LED, RF_SUB_868, RF_2G4_2400, 2xVDIV_MID (5 non-critical)

Board needs manual KiCad GUI finish (~45min) OR order as-is for pad testing.
4-layer board design in progress — should route to 0/0 on first pass.
Parts:
- moved U3 5.39 mm to (4.00, 28.0)
- moved U4 5.00 mm to (8.00, 18.0)
- moved C2 3.61 mm to (10.0, 22.0)
- moved C1 2.83 mm to (10.0, 20.0)
- moved D1 2.00 mm to (6.00, 18.0)
Routing:
- net GND: track 117.3 -> 143.3 mm, vias 1 -> 0
- net GPS_RX: track 0.00 -> 21.9 mm, vias 0 -> 2
- net VCAP: track 6.74 -> 26.5 mm, vias 0 -> 1
- net SPI_SCK: track 12.1 -> 0.00 mm
- net SPI_MOSI: track 0.00 -> 10.8 mm, vias 0 -> 2
- net LR2021_RST: track 59.5 -> 51.2 mm
- net 3V3: track 30.1 -> 35.1 mm, vias 2 -> 3
- net FEM_TX: track 35.2 -> 39.6 mm
- net SPI_NSS: track 16.9 -> 13.9 mm
- net LED_ANODE: track 8.52 -> 9.47 mm
- net SPI_MISO: track 25.5 -> 25.1 mm, vias 3 -> 2
