File: tracker/hardware/output/v8j_krt_ms5611.kicad_pcb (KiCad board)
At the start: 4 copper layers, 55 x 45 mm, 28 parts, among them J1 Prog_Header, J2 Debug_Header, U1 ESP32-C3-WROOM-02, U2 LoRa2021_Gen4, U3 MAX-M10S, U4 TPS7A02, U5 MS5611-01BA

Commit message: fix(hw): v8j U5 MS5611 nets + zone refill -> 0 unconnected, 159/159 DRC errors cleared (5 under-size vias left)
Connections:
- U5 pad 4: I2C_SCL -> +3V3
- U5 pad 5: I2C_SDA -> +3V3
- U5 pad 7: GND -> I2C_SDA
- U5 pad 8: GND -> I2C_SCL
Routing:
- net GND: track 100.9 -> 119.1 mm, vias 14 -> 15
- net EN: track 30.6 -> 48.8 mm
- net I2C_SCL: track 43.8 -> 61.2 mm, vias 2 -> 5
- net I2C_SDA: track 43.5 -> 60.8 mm, vias 2 -> 3
- net +3V3: track 54.8 -> 68.0 mm, vias 8 -> 10
