File: tracker/hardware/schematics/v_c3_flight.kicad_sch (KiCad schematic)
At the start: 22 parts, among them J1 Prog_Header, J2 Debug_Header, U1 ESP32-C3-WROOM-02, U2 LR2021F33, U3 MAX-M10S, U4 TPS7A02, U5 BMP280 (opt)

Commit message: M1: align MS5611 design-backing artifacts (BOM, netlist, generator, schematics)
- v8b BOM/position files now list U5 as MS5611 with Package_LGA:LGA-8_3x5mm_P1.25mm
- flight_board netlist, build script, and regenerated schematic now emit Sensor_Pressure:MS5611-01BA
- top-level v_c3_flight.kicad_sch U5 symbol/value/footprint updated to MS5611-01BA
- hub_schematic stale BMP280-only comment fixed

No active design source file still declares BMP280 as the populated part.
Parts:
- U5: value BMP280 (opt) -> MS5611-01BA; footprint Package_LGA:Bosch_LGA-8_2.5x2.0mm_P0.65mm -> Package_LGA:LGA-8_3x5mm_P1.25mm; symbol Sensor_Pressure:BMP280 -> Sensor_Pressure:MS5611-01BA
Changed lines of the file:
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@@
 	)
 	(symbol
-		(lib_id "Sensor_Pressure:BMP280")
+		(lib_id "Sensor_Pressure:MS5611-01BA")
 		(at 320 60 0)
 		(unit 1)
@@
 			)
 		)
-		(property "Value" "BMP280 (opt)"
+		(property "Value" "MS5611-01BA"
 			(at 0 2.54 0)
 			(effects
@@
 				)
 			)
-		)			(property "Footprint" "Package_LGA:Bosch_LGA-8_2.5x2.0mm_P0.65mm"
+		)			(property "Footprint" "Package_LGA:LGA-8_3x5mm_P1.25mm"
 			(at 0 0 0)
 			(effects
@@
 				(reference "U5")
 				(unit 1)
-				(value "BMP280 (opt)")
-				(footprint "")
-			)
+				(value "MS5611-01BA")
+				(footprint "")
+			)
