File: tracker/hardware/schematics/flight_board/v9_flight.kicad_sch (KiCad schematic)
At the start: 27 parts, among them U1 ESP32-S3-WROOM-1U-N8R8, U2 LoRa2021F33-2G4, U3 LoRa2021_Castellated, U4 SX1280, U5 MAX-M10S, U6 MS5611-01BA, U7 TPS7A02

Commit message: fix(adr): 044a -> 047 (sequential convention) so the numbering gate is green; generator reproduces the artifact
Other:
- note added: "ADR-047 (operator directive 2026-10-07): F33 pin 1 VCC is provisioned for the MODULE MAXIMUM DRAW (1118 mA @ 5.5 V = 6.15 W DC) and is fed from the RAW supercap node (VSCAP, post-BAT54, PRE-LDO) through the ADR-029 D8 pin-1 selector J_VCC. It is NEVER fed through the TPS7A02 (<=300 mA vs 1118 mA = hard failure). Local bulk C_BULK + C_HF, clamp D_CLAMP, rail monitor R_MON1/R_MON2/C_MON -> IO13. Fu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"
- note added: "F33 RAIL PROVISION (ADR-047): pin-1 selector / bulk / clamp / monitor"
- note added: "TODO(unverified) OPEN-15 SUPERCAP CELL ESR + COLD BANK BEHAVIOUR -- ADR-047 3/4: the AVX SCC 3.3 F 2.7 V cell's ESR is NOT in this repository, at 25 C or at -60 C. Every rail-step number in ADR-047 is conditional on the assumed 0.10 Ohm/cell. ADR-029 5 test 4 (<20 mV rail dip during a worst-case burst) is NOT met by scaling this cell family: 16.7 mOhm would need ~12 cells in parallel per series p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"
- note added: "TODO(unverified) OPEN-16 CLAMP SET POINT (D_CLAMP) -- ADR-047 7: the clamp must conduct above the 5.4 V rail top and below the F33's damage threshold, which Rev 1.1 of the datasheet does not publish; the 12-cell array's open-circuit voltage at -60 C is also unmeasured. Part and set point cannot be finalised - do not order a guess."
- note added: "TODO(unverified) OPEN-17 RAIL-MONITOR ADC CHANNEL (U1 pin 21 = IO13) -- ADR-047 6: IO13 is unassigned by the ADR-029 pin plan, and ADR-038 D1 makes Wi-Fi/BT never enabled (CONFIG_ESP_WIFI_ENABLED=n), which is the condition normally attached to ESP32-S3 ADC2 use. Those two facts are the whole basis for putting the monitor there. The ADC channel number and the ADC's required source impedance are NO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"
- note added: "TODO(unverified) OPEN-18 O5 EVIDENCE STILL OPEN -- ADR-029 O5 / ADR-044 7: no 5 V chain demonstrated at >=1.2 A load-step capability, no 3.3 V rail at >=0.60 A transient, no cold supercap or regulator evidence, no ADR-029 5 test 4. ADR-047 sizes for the maximum draw; it does not measure the chain. The BOM freeze stays gated on this."
- note added: "U2 LoRa2021F33-2G4 (433 MHz TX) - VCC PRE-LDO, ADR-047"
- note removed: "ADR-044a (operator directive 2026-10-07): F33 pin 1 VCC is provisioned for the MODULE MAXIMUM DRAW (1118 mA @ 5.5 V = 6.15 W DC) and is fed from the RAW supercap node (VSCAP, post-BAT54, PRE-LDO) through the ADR-029 D8 pin-1 selector J_VCC. It is NEVER fed through the TPS7A02 (<=300 mA vs 1118 mA = hard failure). Local bulk C_BULK + C_HF, clamp D_CLAMP, rail monitor R_MON1/R_MON2/C_MON -> IO13. F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"
- note removed: "F33 RAIL PROVISION (ADR-044a): pin-1 selector / bulk / clamp / monitor"
- note removed: "TODO(unverified) OPEN-15 SUPERCAP CELL ESR + COLD BANK BEHAVIOUR -- ADR-044a 3/4: the AVX SCC 3.3 F 2.7 V cell's ESR is NOT in this repository, at 25 C or at -60 C. Every rail-step number in ADR-044a is conditional on the assumed 0.10 Ohm/cell. ADR-029 5 test 4 (<20 mV rail dip during a worst-case burst) is NOT met by scaling this cell family: 16.7 mOhm would need ~12 cells in parallel per series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"
- note removed: "TODO(unverified) OPEN-16 CLAMP SET POINT (D_CLAMP) -- ADR-044a 7: the clamp must conduct above the 5.4 V rail top and below the F33's damage threshold, which Rev 1.1 of the datasheet does not publish; the 12-cell array's open-circuit voltage at -60 C is also unmeasured. Part and set point cannot be finalised - do not order a guess."
- note removed: "TODO(unverified) OPEN-17 RAIL-MONITOR ADC CHANNEL (U1 pin 21 = IO13) -- ADR-044a 6: IO13 is unassigned by the ADR-029 pin plan, and ADR-038 D1 makes Wi-Fi/BT never enabled (CONFIG_ESP_WIFI_ENABLED=n), which is the condition normally attached to ESP32-S3 ADC2 use. Those two facts are the whole basis for putting the monitor there. The ADC channel number and the ADC's required source impedance are N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"
- note removed: "TODO(unverified) OPEN-18 O5 EVIDENCE STILL OPEN -- ADR-029 O5 / ADR-044 7: no 5 V chain demonstrated at >=1.2 A load-step capability, no 3.3 V rail at >=0.60 A transient, no cold supercap or regulator evidence, no ADR-029 5 test 4. ADR-044a sizes for the maximum draw; it does not measure the chain. The BOM freeze stays gated on this."
- note removed: "U2 LoRa2021F33-2G4 (433 MHz TX) - VCC PRE-LDO, ADR-044a"
Changed lines of the file:
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@@
 			(justify left bottom)
 		)
-	)	(text "ADR-044a (operator directive 2026-10-07): F33 pin 1 VCC is provisioned for the MODULE MAXIMUM DRAW (1118 mA @ 5.5 V = 6.15 W DC) and is fed from the RAW supercap node (VSCAP, post-BAT54, PRE-LDO) through the ADR-029 D8 pin-1 selector J_VCC. It is NEVER fed through the TPS7A02 (<=300 mA vs 1118 mA = hard failure). Local bulk C_BULK + C_HF, clamp D_CLAMP, rail monitor R_MON1/R_MON2/C_MON -> IO13. Full +33 dBm needs >=5.0 V rail; +30 dBm needs >=3.54 V interpolated (ADR-044 S8 table). Firmware must gate TX on the LOADED rail."
+	)	(text "ADR-047 (operator directive 2026-10-07): F33 pin 1 VCC is provisioned for the MODULE MAXIMUM DRAW (1118 mA @ 5.5 V = 6.15 W DC) and is fed from the RAW supercap node (VSCAP, post-BAT54, PRE-LDO) through the ADR-029 D8 pin-1 selector J_VCC. It is NEVER fed through the TPS7A02 (<=300 mA vs 1118 mA = hard failure). Local bulk C_BULK + C_HF, clamp D_CLAMP, rail monitor R_MON1/R_MON2/C_MON -> IO13. Full +33 dBm needs >=5.0 V rail; +30 dBm needs >=3.54 V interpolated (ADR-044 S8 table). Firmware must gate TX on the LOADED rail."
 		(exclude_from_sim no)
 		(at 30.48 24.13 0)
@@
 			(justify left bottom)
 		)
-	)	(text "U2 LoRa2021F33-2G4  (433 MHz TX) - VCC PRE-LDO, ADR-044a"
+	)	(text "U2 LoRa2021F33-2G4  (433 MHz TX) - VCC PRE-LDO, ADR-047"
 		(exclude_from_sim no)
 		(at 182.88 43.18 0)
@@
 			(justify left bottom)
 		)
-	)	(text "F33 RAIL PROVISION (ADR-044a): pin-1 selector / bulk / clamp / monitor"
+	)	(text "F33 RAIL PROVISION (ADR-047): pin-1 selector / bulk / clamp / monitor"
 		(exclude_from_sim no)
 		(at 411.48 43.18 0)
@@
 			(justify left bottom)
 		)
-	)	(text "TODO(unverified) OPEN-15 SUPERCAP CELL ESR + COLD BANK BEHAVIOUR -- ADR-044a 3/4: the AVX SCC 3.3 F 2.7 V cell's ESR is NOT in this repository, at 25 C or at -60 C. Every rail-step number in ADR-044a is conditional on the assumed 0.10 Ohm/cell. ADR-029 5 test 4 (<20 mV rail dip during a worst-case burst) is NOT met by scaling this cell family: 16.7 mOhm would need ~12 cells in parallel per series position."
+	)	(text "TODO(unverified) OPEN-15 SUPERCAP CELL ESR + COLD BANK BEHAVIOUR -- ADR-047 3/4: the AVX SCC 3.3 F 2.7 V cell's ESR is NOT in this repository, at 25 C or at -60 C. Every rail-step number in ADR-047 is conditional on the assumed 0.10 Ohm/cell. ADR-029 5 test 4 (<20 mV rail dip during a worst-case burst) is NOT met by scaling this cell family: 16.7 mOhm would need ~12 cells in parallel per series position."
 		(exclude_from_sim no)
 		(at 30.48 403.86 0)
@@
 			(justify left bottom)
 		)
-	)	(text "TODO(unverified) OPEN-16 CLAMP SET POINT (D_CLAMP) -- ADR-044a 7: the clamp must conduct above the 5.4 V rail top and below the F33's damage threshold, which Rev 1.1 of the datasheet does not publish; the 12-cell array's open-circuit voltage at -60 C is also unmeasured. Part and set point cannot be finalised - do not order a guess."
+	)	(text "TODO(unverified) OPEN-16 CLAMP SET POINT (D_CLAMP) -- ADR-047 7: the clamp must conduct above the 5.4 V rail top and below the F33's damage threshold, which Rev 1.1 of the datasheet does not publish; the 12-cell array's open-circuit voltage at -60 C is also unmeasured. Part and set point cannot be finalised - do not order a guess."
 		(exclude_from_sim no)
 		(at 30.48 407.67 0)
@@
 			(justify left bottom)
 		)
-	)	(text "TODO(unverified) OPEN-17 RAIL-MONITOR ADC CHANNEL (U1 pin 21 = IO13) -- ADR-044a 6: IO13 is unassigned by the ADR-029 pin plan, and ADR-038 D1 makes Wi-Fi/BT never enabled (CONFIG_ESP_WIFI_ENABLED=n), which is the condition normally attached to ESP32-S3 ADC2 use. Those two facts are the whole basis for putting the monitor there. The ADC channel number and the ADC's required source impedance are NOT in this repository, and the pin plan has not yet been amended to record the assignment."
+	)	(text "TODO(unverified) OPEN-17 RAIL-MONITOR ADC CHANNEL (U1 pin 21 = IO13) -- ADR-047 6: IO13 is unassigned by the ADR-029 pin plan, and ADR-038 D1 makes Wi-Fi/BT never enabled (CONFIG_ESP_WIFI_ENABLED=n), which is the condition normally attached to ESP32-S3 ADC2 use. Those two facts are the whole basis for putting the monitor there. The ADC channel number and the ADC's required source impedance are NOT in this repository, and the pin plan has not yet been amended to record the assignment."
 		(exclude_from_sim no)
 		(at 30.48 411.48 0)
@@
 			(justify left bottom)
 		)
-	)	(text "TODO(unverified) OPEN-18 O5 EVIDENCE STILL OPEN -- ADR-029 O5 / ADR-044 7: no 5 V chain demonstrated at >=1.2 A load-step capability, no 3.3 V rail at >=0.60 A transient, no cold supercap or regulator evidence, no ADR-029 5 test 4. ADR-044a sizes for the maximum draw; it does not measure the chain. The BOM freeze stays gated on this."
+	)	(text "TODO(unverified) OPEN-18 O5 EVIDENCE STILL OPEN -- ADR-029 O5 / ADR-044 7: no 5 V chain demonstrated at >=1.2 A load-step capability, no 3.3 V rail at >=0.60 A transient, no cold supercap or regulator evidence, no ADR-029 5 test 4. ADR-047 sizes for the maximum draw; it does not measure the chain. The BOM freeze stays gated on this."
 		(exclude_from_sim no)
 		(at 30.48 415.29 0)

Commit message: feat(v9 hub): add the FOUR wing-mount interfaces (ADR-048 / ADR-046)
The v9 hub is a 3D assembly: one hub + four identical wings soldered on at
90 deg.  The hub had NO wing interface; the wing tab (4 pads, ADR-046 s2.1)
and the hub-side requirement (docs/WING-TO-HUB-SOCKET-SPEC.md) were already
fixed, so this lands the hub side.

Generator (v9 target only; the C3 target's output is byte-identical):
  * balloon_flight_v9:WING_SOCKET_4P symbol - 4 pins, names from ADR-046 s2.1
    (SOLAR_P / GND / RF_FEED / SOLAR_N), all passive: a hand-soldered land set
    with no driver, so no PA/RF/power termination is asserted anywhere.
  * J_W1..J_W4 - the four interfaces, one per hub edge, 90 deg apart.
  * Hub series stack implemented per ADR-046 s2.3 / socket spec s3.1:
    W1_SOLAR_P -> BAT54 (D1) -> supercap; the hub links W1_SOLAR_N==W2_SOLAR_P,
    W2_SOLAR_N==W3_SOLAR_P, W3_SOLAR_N==W4_SOLAR_P as one node each;
    W4_SOLAR_N = stack bottom = GND; every interface GND land on GND.
  * D_BP1..D_BP4 - the mandated DNP bypass Schottky per interface (socket
    spec s5), cathode to W<n>_SOLAR_P.
  * pin 3 (W<n>_RF) is left with NO net and NO no_connect flag: ADR-046 s2.4
    and socket spec s3.2 say the v9 RF land is an isolated provision.  It
    therefore shows up as 4 new pin_not_connected ERC errors - recorded, not
    silenced (OPEN-21).
  * OPEN-12 (solar input source) closed; OPEN-20..OPEN-24 opened for the land
    datum / edge clearance conflict, the unnetted RF lands, the hub stack-up,
    the conflicting assembly-orientation records, and the unmeasured hand
    solder-joint dimensions.

Real footprint (not a generic pin header):
  tracker/hardware/footprints/tracker_mechanical.pretty/Wing_Tab_4P.kicad_mod
  - 8 lands per interface (4 per face, both outer layers), 4.0 x 1.2 mm,
  pitch 1.8 mm, 0.9 x 6.0 mm Edge.Cuts slot, spec keep-outs (slot +1.0 mm,
  courtyard 1.5 mm from the land row) and spec silkscreen (W / 1 / 4 / 90 /
  slot-axis tick), with the 1.0 mm coppe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
Parts:
- removed U6: MS5611-01BA, Package_LGA:LGA-8_3x5mm_P1.25mm, symbol Sensor_Pressure:MS5611-01BA
- added D_BP1, D_BP2, D_BP3, D_BP4: BAT54 (DNP), Diode_SMD:D_SOD-323, symbol Device:D_Schottky
- added J_W1: WING_SOCKET_4P (hub wing interface 1), Tracker_Mechanical:Wing_Tab_4P, symbol balloon_flight_v9:WING_SOCKET_4P
- added J_W2: WING_SOCKET_4P (hub wing interface 2), Tracker_Mechanical:Wing_Tab_4P, symbol balloon_flight_v9:WING_SOCKET_4P
- added J_W3: WING_SOCKET_4P (hub wing interface 3), Tracker_Mechanical:Wing_Tab_4P, symbol balloon_flight_v9:WING_SOCKET_4P
- added J_W4: WING_SOCKET_4P (hub wing interface 4), Tracker_Mechanical:Wing_Tab_4P, symbol balloon_flight_v9:WING_SOCKET_4P
- added U7: TPS7A02, Package_TO_SOT_SMD:SOT-23-5, symbol balloon_flight_v9:TPS7A0233
- U6: renamed from U7; value TPS7A02 -> MS5611-01BA; footprint Package_TO_SOT_SMD:SOT-23-5 -> Package_LGA:LGA-8_3x5mm_P1.25mm; symbol balloon_flight_v9:TPS7A0233 -> Sensor_Pressure:MS5611-01BA
Connections:
- net +3V3: now also U6.1 (VDD), U7.5 (OUT); no longer U6.5 (OUT)
- net GND: now also U6.3 (GND), D_BP4.2 (A), J_W1.2 (GND), J_W2.2 (GND), J_W3.2 (GND), J_W4.2 (GND), J_W4.4 (SOLAR_N), U7.2 (GND); no longer U6.2 (GND)
- net I2C_SCL: now also U6.8 (SCLK)
- net I2C_SDA: now also U6.7 (SDI/SDA)
- net VSCAP: now also U7.1 (IN), U7.3 (EN); no longer U6.1 (IN), U6.3 (EN)
- net at U6.4 (CSB): now also U6.5 (CSB)
- net SOLAR_IN renamed W1_SOLAR_P
- net W1_SOLAR_P: now also D_BP1.1 (K), J_W1.1 (SOLAR_P)
- new net W1_SOLAR_N: D_BP1.2 (A), D_BP2.1 (K), J_W1.4 (SOLAR_N), J_W2.1 (SOLAR_P)
- new net W2_SOLAR_N: D_BP2.2 (A), D_BP3.1 (K), J_W2.4 (SOLAR_N), J_W3.1 (SOLAR_P)
- new net W3_SOLAR_N: D_BP3.2 (A), D_BP4.1 (K), J_W3.4 (SOLAR_N), J_W4.1 (SOLAR_P)
Other:
- note added: "ADR-046 + ADR-048 (wing interface, Status PROPOSED - not human-accepted): the v9 hub carries FOUR wing-mount interfaces at 90 deg spacing, J_W1..J_W4. Each is one socket land set: 4 copper lands per face on BOTH outer layers = 8 lands per interface, land 4.0 x 1.2 mm, pitch 1.8 mm, insertion depth 6.0 mm. Net order 1 SOLAR_P / 2 GND / 3 RF_FEED (v9 provision, NO NET) / 4 SOLAR_N. Series stack wir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"
- note added: "BALLOON v9 TRI-BAND FLIGHT BOARD - DESIGN-INTENT schematic from the v9 decision records (ADR-029/034/035/036-043, ADR-044/044a/045/046/047/048). NOT derived from a PCB."
- note added: "FOUR WING INTERFACES at 90 deg (ADR-046 / ADR-048): 4 lands per face x 2 faces = 8 lands each, 4.0 x 1.2 mm, pitch 1.8 mm; 1 SOLAR_P / 2 GND / 3 RF (NO NET on v9) / 4 SOLAR_N + 4 DNP bypass Schottky"
- note added: "TODO(unverified) OPEN-12 SOLAR INPUT SOURCE (CLOSED by ADR-048) -- ADDRESSED: the 4-wing x 3-cell solar array input IS the four wing-mounted interfaces J_W1..J_W4 added by ADR-048 (ADR-046 s1/s2.3 + socket spec s1). The net that used to be a 1-pad `SOLAR_IN` (D1 anode only) is now W1_SOLAR_P and carries J_W1 pad 1 as the stack top. What is NOT closed: the wing-side array-coverage / bypass re-budg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"
- note added: "TODO(unverified) OPEN-20 HUB-SIDE LAND DATUM + EDGE CLEARANCE (ADR-048 D-1) -- The socket spec s2 gives the land row's along-insertion offset twice and incompatibly: 'Land centre offset from the hub's outer edge 1.0 mm inboard' versus its own parenthetical 'lands span 0.0...4.0 mm from the edge' (centre 2.0 mm) - a 1.0 mm self-contradiction - while ADR-046 s2.2 fixes copper-to-board-edge clearanc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"
- note added: "TODO(unverified) OPEN-21 W<n>_RF PROVISION LANDS ARE UNNETTED (4 NEW ERC ERRORS, BY DESIGN) -- ADR-046 s2.4 and socket spec s3.2 mandate that each interface's pad 3 (RF_FEED) keeps its copper land but carries NO NET on v9, and explicitly say 'Do not tie it to GND'. The sheet therefore leaves J_W1..J_W4 pin 3 floating and does NOT add a no_connect flag: a no_connect would assert a termination deci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"
- note added: "TODO(unverified) OPEN-22 HUB v9 STACK-UP / SLOT KEEP-OUT / FAB TOLERANCE -- Socket spec s8 items 1-4 are all still open: the hub's actual component keep-out at the slot (which owns whether the 6.0 mm slot depth is legally routable and whether the slot keep-out may exceed the +1.0 mm of s4); JLCPCB's routed-slot width tolerance (0.9 mm +/-0.10 mm is an ASSUMPTION, ADR-046 s4.3); the v9 hub layer c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"
- note added: "TODO(unverified) OPEN-23 ASSEMBLY ORIENTATION OF THE WING AT THE HUB (CONFLICTING RECORDS) -- Socket spec s1 says the wing's long axis is 'perpendicular to the hub plane' and then, in the next sentence, that wings 1-2 are 'horizontal' in the hub plane (and 3-4 inclined ~30 deg below it); ADR-046 s4.1 says '90 deg to the hub plane, wing plane normal to the hub plane'. The two readings cannot both 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"
- note added: "TODO(unverified) OPEN-24 HAND-SOLDER JOINT DIMENSIONS NOT MEASURED -- The v9 hub does not exist and neither the wing tab's nor the cells' real contact geometry has been measured: ADR-046 s7 item 1 files the 52 x 19 mm cell tab geometry as TODO(unverified), ADR-046 s7 item 8 files the tab fillet's structural adequacy under the ~176 mm cantilever as unanalysed, and ADR-046 s4.3 flags that a slot wh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"
- note removed: "BALLOON v9 TRI-BAND FLIGHT BOARD - DESIGN-INTENT schematic from the v9 decision records (ADR-029/034/035/036-043, ADR-044/044a/045). NOT derived from a PCB."
- note removed: "TODO(unverified) OPEN-12 SOLAR INPUT SOURCE -- The 4-wing x 3-cell solar array input connector is not in the v9 component list; SOLAR_IN has only the D1 anode end so far."
