File: tracker/hardware/schematics/flight_board/v9_flight.kicad_sch (KiCad schematic)
At the start: 35 parts, among them U1 ESP32-S3-WROOM-1U-N8R8, U2 LoRa2021F33-2G4, U3 LoRa2021_Castellated, U4 SX1280, U5 MAX-M10S, U6 MS5611-01BA, U7 TPS7A02

Commit message: feat(v9-sch): implement the locked array + cut topology (ADR-051/053/054)
Implements, in the v9 design-intent generator (build_flight_sch.py, v9 target),
the four electrical decisions that were already merged.  Regenerated artifacts:
v9_flight.kicad_sch, v9_flight.net, v9_flight-erc.rpt,
v9_lib/balloon_flight_v9.kicad_sym.

1. HUB ARRAY AS AN ELECTRICALLY INDEPENDENT SERIES STRING (ADR-051 s2.1 as
   amended, ADR-054 s2.1).  It gets its OWN nets HUB_PV_P / HUB_PV_MID<n> /
   HUB_PV_N and its OWN converter input (U_HUB_CVT); it is never in series
   with, and never a tap on, the wing chain - the only shared node is GND,
   through the converter's ground pin.  Cells PVA<n> per ADR-051 s2.1.1.
   The cell count is a DOCUMENTED PLACEHOLDER (V9_HUB_ARRAY_CELLS = 2,
   ADR-051 s2.2's recommended H2): the hub outline is a form-factor decision
   owned by another task (ADR-051 s2.3), and the count, the mounting plane and
   the harvester part are OPEN (OPEN-26).

2. THE PER-INTERFACE BYPASS DIODES D_BP1..D_BP4 ARE POPULATED AND RE-RATED
   (ADR-051 s2.7, ADR-053 s2.2 as amended by ADR-054 s3.2).
   BAT54 (DNP, 200 mA / 30 V, SOD-323) -> SS24 (2 A / 40 V, SMA), DNP cleared,
   still HUB-SIDE across W<n>_SOLAR_P (K) / W<n>_SOLAR_N (A).  The WHY is
   recorded in the generator comments and on the sheet: a cut jettisons the
   wing and everything soldered to it, so only a HUB-side diode can restore
   the broken path; and a failed cell - and every post-cut path - is a
   PERMANENT CONTINUOUS bypass condition, not a shading transient, so the
   200 mA part is disqualified, and 30 V cannot clear the ~9.58 V cold
   open-circuit stack.  The minimal per-hub-cell provision D_HUB<n> is added
   so the fail-closed bypass checker can reach a DETERMINATE answer for the
   hub cells as well; the hub's per-cell/per-group granularity stays OPEN
   (OPEN-27).

3. CUT-SENSE ON THE RESERVED W<n>_RF (RF_FEED) PIN (ADR-051 s2.6).  J_W<n>
   pad 3 now carries CUT_SENSE_W<n> - the nichrome cutter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
Parts:
- removed ANT3: U.FL_2G4_RX, Connector_Coaxial:U.FL_Molex_MCRF_73412-0110_Vertical, symbol Connector:Conn_Coaxial
- removed ANT4: U.FL_GNSS_L1, Connector_Coaxial:U.FL_Molex_MCRF_73412-0110_Vertical, symbol Connector:Conn_Coaxial
- added C_BULK: 100uF, Capacitor_SMD:C_1206_3216Metric, symbol Device:C
- added D_HUB1, D_HUB2: SS24, Diode_SMD:D_SMA, symbol Device:D_Schottky
- added J_VCC: F33_VCC_SEL (5V raw | 3V3), Jumper:SolderJumper-3_P1.3mm_Open_RoundedPad1.0x1.5mm, symbol balloon_flight_v9:F33_VCC_SEL
- added PVA1, PVA2: SolarCell_78x39mm, symbol balloon_flight_v9:PVA_CELL
- added U_CUT1, U_CUT2, U_CUT3, U_CUT4: latched cut driver + cut-sense (part TODO(unverif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, symbol balloon_flight_v9:CUT_CHANNEL
- added U_HUB_CVT: HUB_PV input (part TODO(unverified)), symbol balloon_flight_v9:HUB_CONVERTER
- ANT3: renamed from J_VCC; value F33_VCC_SEL (5V raw | 3V3) -> U.FL_2G4_RX; footprint Jumper:SolderJumper-3_P1.3mm_Open_RoundedPad1.0x1.5mm -> Connector_Coaxial:U.FL_Molex_MCRF_73412-0110_Vertical; symbol balloon_flight_v9:F33_VCC_SEL -> Connector:Conn_Coaxial
- ANT4: renamed from C_BULK; value 100uF -> U.FL_GNSS_L1; footprint Capacitor_SMD:C_1206_3216Metric -> Connector_Coaxial:U.FL_Molex_MCRF_73412-0110_Vertical; symbol Device:C -> Connector:Conn_Coaxial
- D_BP1, D_BP2, D_BP3, D_BP4: value BAT54 (DNP) -> SS24; footprint Diode_SMD:D_SOD-323 -> Diode_SMD:D_SMA; now fitted
Connections:
- net +3V3: now also J_VCC.3 (B_3V3); no longer ANT3.3 (B_3V3)
- net ANT3_2G4_RX: now also ANT3.1 (In)
- net ANT4_GNSS_L1: now also ANT4.1 (In)
- net F33_VCC: now also C_BULK.1, J_VCC.2 (COM); no longer ANT3.2 (COM), ANT4.1
- net GND: now also ANT3.2 (Ext), C_BULK.2, U_CUT1.2 (GND), U_CUT2.2 (GND), U_CUT3.2 (GND), U_CUT4.2 (GND), U_HUB_CVT.2 (GND)
- net VSCAP: now also J_VCC.1 (A_VSCAP), U_CUT1.1 (VSCAP), U_CUT2.1 (VSCAP), U_CUT3.1 (VSCAP), U_CUT4.1 (VSCAP); no longer ANT3.1 (A_VSCAP)
- net CUT_SENSE_W4: now reaches J_W4.3 (RF_FEED)
- net CUT_SENSE_W4: now also U_CUT4.3 (CUT_W)
- net CUT_SENSE_W2: now reaches J_W2.3 (RF_FEED)
- net CUT_SENSE_W2: now also U_CUT2.3 (CUT_W)
- net CUT_SENSE_W3: now reaches J_W3.3 (RF_FEED)
- net CUT_SENSE_W3: now also U_CUT3.3 (CUT_W)
- net CUT_SENSE_W1: now reaches J_W1.3 (RF_FEED)
- net CUT_SENSE_W1: now also U_CUT1.3 (CUT_W)
- new net HUB_PV_MID1: D_HUB1.2 (A), D_HUB2.1 (K), PVA1.2 (N), PVA2.1 (P)
- new net HUB_PV_N: D_HUB2.2 (A), PVA2.2 (N), U_HUB_CVT.3 (PV_N)
- new net HUB_PV_P: D_HUB1.1 (K), PVA1.1 (P), U_HUB_CVT.1 (PV_P)
Other:
- note added: "ADR-051 s2.1 - THE HUB ARRAY IS AN INDEPENDENT SERIES STRING. It has its OWN nets (HUB_PV_P positive, HUB_PV_MID<n> interior, HUB_PV_N negative) and its OWN converter/harvester input (U_HUB_CVT), and it is NEVER in series with, and never a tap on, the wing chain - the ONLY node it may share with the wing system is GND, and only through the converter's ground pin. If it were wired into the wing ch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"
- note added: "ADR-051 s2.5 decision item 5 - THE CUT DRIVE MUST BE A LATCHED ONE-SHOT, one per wing (U_CUT1..U_CUT4). Cutting is IRREVERSIBLE, and a level-sensitive driver can RE-FIRE an already-fired channel on a reset, a brown-out, a firmware retry or a floating gate - each fire costing ~2.59 J of the bank's 16.63 J usable energy at the exact moment the bank matters (ADR-051 s2.5.1). The mandate: a firmware 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"
- note added: "ADR-051 s2.6 - THE RESERVED RF_FEED LAND IS NOW THE PER-WING CUT-SENSE / CUTTER LINE. J_W<n> pad 3 carries CUT_SENSE_W<n>, which does the nichrome cutter drive AND the continuity sense on ONE conductor plus the shared ground - four independently controllable cutters at ZERO connector cost, because the land and the position were already paid for. Netting it closes the four pin_not_connected ERC er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"
- note added: "ADR-051 s2.7 / ADR-054 s2.2+s3.2 - THE PER-INTERFACE BYPASS DIODES ARE POPULATED AND RE-RATED, AND THEY SIT HUB-SIDE. D_BP1..D_BP4 bridge each wing interface (W<n>_SOLAR_P cathode -> W<n>_SOLAR_N anode) and are now SS24 = 2 A / 40 V on an SMA land, not DNP BAT54 = 200 mA / 30 V on SOD-323. WHY HUB-SIDE: a cut jettisons the wing AND every part soldered to it, so only a HUB-side diode can bridge th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"
- note added: "BALLOON v9 TRI-BAND FLIGHT BOARD - DESIGN-INTENT schematic from the v9 decision records (ADR-029/034/035/036-043, ADR-044/044a/045/046/047/048/049/050/051/052/053/054). NOT derived from a PCB."
- note added: "FOUR WING INTERFACES at 90 deg (ADR-046 / ADR-048): 4 lands per face x 2 faces = 8 lands each, 4.0 x 1.2 mm, pitch 1.8 mm; 1 SOLAR_P / 2 GND / 3 RF = CUT_SENSE_W<n> (ADR-051 s2.6) / 4 SOLAR_N + 4 POPULATED bypass Schottky (SS24, 2 A / 40 V)"
- note added: "INDEPENDENT HUB ARRAY (ADR-051 s2.1) + 4 LATCHED CUT CHANNELS (s2.5/s2.6)"
- note added: "TODO(unverified) OPEN-21 W<n>_RF PROVISION LANDS (CLOSED by ADR-051 s2.6) -- ADDRESSED: ADR-046 s2.4 / socket spec s3.2 left each interface's pad 3 (RF_FEED) with its copper land but NO net, and explicitly said 'Do not tie it to GND'; that produced 4 pin_not_connected ERC errors by design. ADR-051 s2.6 now NETS that land as CUT_SENSE_W<n>, so those 4 errors are CLOSED at zero connector cost. The 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"
- note added: "TODO(unverified) OPEN-25 CUT-SENSE GPIO / DIVIDER AND THE WING RE-SPIN -- ADR-051 s2.6 fixes the MECHANISM (per-wing CUT_SENSE_W<n> on the reserved RF_FEED land) but NOT the GPIO count: four dedicated GPIOs, or one GPIO plus a 4:1 analogue mux / resistor-ladder encoding, are both compatible and the sense divider values are not chosen. GPIO budget is the constraint (ADR-029 free-GPIO audit; OPEN-1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"
- note added: "TODO(unverified) OPEN-26 HUB ARRAY: CELL COUNT, MOUNTING PLANE, HARVESTER, OUTLINE -- ADR-051 s2.1's independence invariant is IMPLEMENTED on this sheet, but the array's PARAMETERS are not: the cell count (H2 = 2 recommended / H3 = 3 fallback), the mounting plane (vertical 0.3051 vs horizontal 0.1865 day-mean - load-bearing for the area), the converter/harvester part and its peak-input-power rati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"
- note added: "TODO(unverified) OPEN-27 HUB-ARRAY BYPASS GRANULARITY (PER-CELL vs PER-GROUP) -- ADR-051 s2.2 places the hub cells on the hub and says they 'need their own diodes'; ADR-054 s4.5 explicitly leaves the hub array's per-cell-over-per-group trade OPEN. This sheet carries the MINIMAL per-cell provision (D_HUB<n>, one SS24 across each hub cell) because scripts/bypass_diode_check.py requires every solar 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"
- note added: "TODO(unverified) OPEN-28 CUT-DRIVER LATCH TOPOLOGY AND ITS PART -- ADR-051 s2.5.1 mandates a LATCHED one-shot with a persistent NVS fired flag per channel plus a hardware series arming gate, but names no part: the IRLML2502 in the repo's own precedent is the switch, not the latch. U_CUT1..U_CUT4 are PROVISION symbols whose pin set (VSCAP / GND / the wing RF_FEED line) is fixed and whose internals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"
- note removed: "BALLOON v9 TRI-BAND FLIGHT BOARD - DESIGN-INTENT schematic from the v9 decision records (ADR-029/034/035/036-043, ADR-044/044a/045/046/047/048). NOT derived from a PCB."
- note removed: "FOUR WING INTERFACES at 90 deg (ADR-046 / ADR-048): 4 lands per face x 2 faces = 8 lands each, 4.0 x 1.2 mm, pitch 1.8 mm; 1 SOLAR_P / 2 GND / 3 RF (NO NET on v9) / 4 SOLAR_N + 4 DNP bypass Schottky"
- note removed: "TODO(unverified) OPEN-21 W<n>_RF PROVISION LANDS ARE UNNETTED (4 NEW ERC ERRORS, BY DESIGN) -- ADR-046 s2.4 and socket spec s3.2 mandate that each interface's pad 3 (RF_FEED) keeps its copper land but carries NO NET on v9, and explicitly say 'Do not tie it to GND'. The sheet therefore leaves J_W1..J_W4 pin 3 floating and does NOT add a no_connect flag: a no_connect would assert a termination deci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"

Commit message: feat(hw): v9 provision for the LR2021 on-chip NTC temp-comp loop (ADR-058)
Adds the NTC thermistor and its series/bias resistor to the v9 design-intent
schematic THROUGH its generator (build_flight_sch.py, v9 target), so the tree
stays reproducible from the generator.

Parts added (BOTH DNP, reason recorded on the sheet and in the netlist note):
  R_NTC1  Device:R                  - series/bias resistor, VTCXO/VNTC rail to the
                                      sense node; value TODO(unverified), it sets
                                      SetNtcParams ntc_r_ratio (DS 2.2 Table 6-70)
  TH_NTC1 Device:Thermistor_NTC     - the NTC, sense node to GND; part/R25/beta
                                      TODO(unverified) (ADR-058 D4)
  nets: VTCXO_VNTC = {U3.13, R_NTC1.1}; NTC_SENSE = {R_NTC1.2, TH_NTC1.1};
        TH_NTC1.2 -> GND

DNP because of the named blocker (ADR-058 D6 / OPEN-29): on the OWNED bare NiceRF
module the chip's NTC sense input (chip pin 3) has no castellation - the vendor pin
table docs/assets/lr2021/LoRa2021-Module-Datasheet-V1.3.pdf 7 enumerates all 18 pads
and the only oscillator pad is 13 = VTCXO - so NTC_SENSE has no path back to the chip
and the loop cannot be closed. The land costs nothing (there is no v9 hub PCB yet) and
a module that does break the pin out closes the loop at zero respin cost.

Also: V9_BARE_PINS pad 13 renamed PAD13_?? -> VTCXO, a naming correction with the
vendor pin-table source (ADR-058 s1.3); OPEN-5 updated (pads 16/17 stay open).
Four new TODO(unverified) notes: OPEN-29 (module pin break-out), OPEN-30 (NTC part +
cold rating vs the -60 degC case), OPEN-31 (SetNtcParams values), OPEN-32 (F33 PA
self-heating vs a nearby NTC).

Gate deltas (baseline e989c01 -> this commit):
  kicad-cli sch erc        24 errors -> 23 errors (0 warnings), all
                           pin_not_connected: ONE error CLOSED (U3 pad 13 now netted
                           on VTCXO_VNTC) and NO new error added.
  scripts/hub_array_topology_c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
Parts:
- removed ANT4: U.FL_GNSS_L1, Connector_Coaxial:U.FL_Molex_MCRF_73412-0110_Vertical, symbol Connector:Conn_Coaxial
- removed D_HUB1: SS24, Diode_SMD:D_SMA, symbol Device:D_Schottky
- added J_VCC: F33_VCC_SEL (5V raw | 3V3), Jumper:SolderJumper-3_P1.3mm_Open_RoundedPad1.0x1.5mm, symbol balloon_flight_v9:F33_VCC_SEL
- added R_NTC1: TODO(unverified) (sets ntc_r_ratio), Resistor_SMD:R_0402_1005Metric, symbol Device:R
- added TH_NTC1: TODO(unverified) (NTC, R25/beta TODO), Resistor_SMD:R_0402_1005Metric, symbol Device:Thermistor_NTC
- added U_HUB_CVT: HUB_PV input (part TODO(unverified)), symbol balloon_flight_v9:HUB_CONVERTER
- ANT4: renamed from J_VCC; value F33_VCC_SEL (5V raw | 3V3) -> U.FL_GNSS_L1; footprint Jumper:SolderJumper-3_P1.3mm_Open_RoundedPad1.0x1.5mm -> Connector_Coaxial:U.FL_Molex_MCRF_73412-0110_Vertical; symbol balloon_flight_v9:F33_VCC_SEL -> Connector:Conn_Coaxial
- D_HUB1: renamed from U_HUB_CVT; value HUB_PV input (part TODO(unverified)) -> SS24; footprint (none) -> Diode_SMD:D_SMA; symbol balloon_flight_v9:HUB_CONVERTER -> Device:D_Schottky
Connections:
- net +3V3: now also J_VCC.3 (B_3V3); no longer ANT4.3 (B_3V3)
- net ANT4_GNSS_L1: now also ANT4.1 (In)
- net F33_VCC: now also J_VCC.2 (COM); no longer ANT4.2 (COM)
- net GND: now also ANT4.2 (Ext), TH_NTC1.2, U_HUB_CVT.2 (GND); no longer D_HUB1.2 (GND)
- net HUB_PV_MID1: now also D_HUB1.2 (A)
- net HUB_PV_N: now also U_HUB_CVT.3 (PV_N); no longer D_HUB1.3 (PV_N)
- net HUB_PV_P: now also U_HUB_CVT.1 (PV_P)
- net VSCAP: now also J_VCC.1 (A_VSCAP); no longer ANT4.1 (A_VSCAP)
- net VTCXO_VNTC: now reaches U3.13 (VTCXO)
- net VTCXO_VNTC: now also R_NTC1.1
- new net NTC_SENSE: R_NTC1.2, TH_NTC1.1
Other:
- note added: "LR2021 ON-CHIP NTC TEMP-COMP PROVISION (ADR-058) - R_NTC1 + TH_NTC1, BOTH DNP: the chip's NTC sense pin (chip pin 3) is NOT broken out on the owned bare NiceRF module (OPEN-29 / ADR-058 D6)"
- note added: "TODO(unverified) OPEN-29 NTC PROVISION: THE MODULE PIN BREAK-OUT (ADR-058 D6, THE BLOCKER) -- Whether the LR2021 chip's NTC sense input (chip pin 3, 'Negative Temperature Coefficient (NTC) resistor connection', DS 2.2 Table 2-1) is broken out on the OWNED bare NiceRF module. EVIDENCE IN HAND SAYS NO: the vendor pin table (docs/assets/lr2021/LoRa2021-Module-Datasheet-V1.3.pdf s7) enumerates ALL 18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"
- note added: "TODO(unverified) OPEN-30 NTC PART SELECTION AND ITS COLD RATING (ADR-058 D4/OPEN-2) -- TH_NTC1's part is NOT chosen. Required in this order: (1) read R25 and beta from the chosen part's own datasheet - they set SetNtcParams ntc_beta ('NTC temperature in 2 Kelvin/lsb', DS 2.2 Table 6-70) and, with R_NTC1, ntc_r_ratio; (2) CHECK THE COLD RATING against the -60 degC design case, with the same rigour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"
- note added: "TODO(unverified) OPEN-31 SetNtcParams VALUES NOT CHARACTERISED (ADR-058 D4) -- The three SetNtcParams inputs are TODO(unverified) and must NOT be invented: ntc_r_ratio (10 bits with 9 fractional bits, the ratio of the bias resistor to the NTC at 25 degC), ntc_beta (2 K/lsb) and delay (first-order time delay coefficient) - DS 2.2 Table 6-70. They must be derived from the POPULATED part + bias resi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"
- note added: "TODO(unverified) OPEN-32 F33 PA SELF-HEATING vs A NEARBY NTC (ADR-058 D3) -- Whether the F33's 2 W PA self-heating perturbs a nearby NTC has NOT been measured (TODO(unverified)). ADR-058 D3 is the siting RULE that this open item exists to protect: the NTC must be thermally coupled to the radio's XTAL / XOSC node and must NOT be sited where a self-heating neighbour dominates its reading (the F33 P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"
- note added: "TODO(unverified) OPEN-5 BARE-MODULE PAD FUNCTIONS (U3 pins 13,16,17) -- PAD13/PAD16/PAD17 functions were unverified (v8i audit: DECLARED_GAP). PARTLY CLOSED by ADR-058 s1.3: pad 13 = VTCXO - the vendor pin table docs/assets/lr2021/LoRa2021-Module-Datasheet-V1.3.pdf s7 enumerates all 18 pads and names pad 13 'VTCXO', O, 'Can provide power for an external TCXO', so the generator's placeholder 'PAD1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"
- note removed: "TODO(unverified) OPEN-5 BARE-MODULE PAD FUNCTIONS (U3 pins 13,16,17) -- PAD13/PAD16/PAD17 functions are unverified (v8i audit: DECLARED_GAP)."

Commit message: sch(v9): close 4 open pin_not_connected from landed records; document the rest
ERC 23 -> 19 errors, all pin_not_connected, 0 warnings. The generator still
regenerates BYTE-IDENTICALLY (v9_flight.kicad_sch sha256 c7a51a51...), and
check_sch_gates.py v9 passes - which checks the generator's own invariants, NOT
electrical correctness. Headline statement: generated + deterministic + ERC 19
errors (was 23).

Closed (4), each with its source:
- U6.2 (PS) and U6.6 (SDO) -> GND; U6.4 (CSB) -> +3V3, on the precedent of the
  frozen tracker/hardware/output/v8j_krt_ms5611.kicad_pcb: SAME
  Package_LGA:LGA-8_3x5mm_P1.25mm footprint, same I2C mode (pads 7/8 =
  I2C_SDA/I2C_SCL, exactly this sheet's U6 7/8), pads 2/4/6 = GND/+3V3/GND.
  The register had only rejected the v8i board, whose barometer is a DIFFERENT
  2.5x2.5 mm footprint. The exported netlist now matches v8j's pad nets
  exactly (1,4,5 = +3V3; 2,3,6 = GND; 7,8 = I2C).
- U1.19 (IO11 / F33_DIO5) -> no-connect: the F33 module has NO DIO5 pad (its
  18-pad table, quoted in-repo at ADR-059 s1.3) and its front-end DIOs are
  internal and written into the chip over SPI, not brought to MCU GPIOs
  (docs/F33-MODULE-PLAN.md; docs/LR2021-LESSONS-2026-09.md). No net invented.

Recorded, NOT silenced - every remaining open pin now names the decision that
must land AND its owner:
- OPEN-1/2 (U4 SX1280 supply + RFIO): ADR-060 s5 re-files these as unfixed;
  ADR-047 prose and docs/POWER-BUDGET-V9-D2BE.md s2 conflict on the 3.3 V rail.
- OPEN-3/4/5 (bare-module NSS/BUSY/RESET/IRQ, sub-GHz ANT, pad functions),
  OPEN-8 (MAX-M10S VIO_SEL/~SAFEBOOT - verified un-netted on the frozen v8i
  board), OPEN-9 (TPS7A02 pin 4), OPEN-10 (ESP32-S3 EN + USB), OPEN-14
  (IO12/IO47/IO48): owner = the ADR-108 pin-plan revision.
- U3.16/U3.17 renamed PAD16_??/PAD17_?? -> DIO8/DIO7 - a NAMING correction with
  a source (vendor pin table s7 + docs/inventory.md line 28); connectivity
  unchanged, the MCU assignment stays OPEN-5.

The MS5611 symbol is re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
Parts:
- U6: symbol Sensor_Pressure:MS5611-01BA -> balloon_flight_v9:MS5611_BARO
Connections:
- net +3V3: now also U6.4 (CSB), U6.5 (CSB)
- net GND: now also U6.2 (PS), U6.6 (SDO)
- no-connect marks 12 -> 13
Other:
- note added: "TODO(unverified) OPEN-1 SX1280 SUPPLY (U4 pins 1,2) -- SX1280 VDD_IN/VDD_IO rail not fixed by any record and the Semtech datasheet is unreachable here. Left open deliberately. ADR-060 s5 (2026-10-07) RE-FILES this as unfixed, which is why it stays open. The conflict to resolve: ADR-047 states the 3.3 V rail also carries the SX1280, and docs/POWER-BUDGET-V9-D2BE.md s2 lists both SX1280 states on t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"
- note added: "TODO(unverified) OPEN-10 ESP32-S3 EN and USB (U1 pins 3,13,14) -- Module EN strap and the USB_D-/USB_D+ pads have no v9 connector or recorded tie-off. The ADR-029 pin plan calls USB-Serial-JTAG the assumed debug path, so these are not unused - they lack a termination. The reset RC is also absent from the v9 BOM (docs/coordination/SCHEMATIC-PLAN-3VARIANTS.md 5 item 2). ADR-108 assigns the FUNCTION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"
- note added: "TODO(unverified) OPEN-14 UNASSIGNED ESP32-S3 GPIO (U1 pins 20,24,25 = IO12, IO47, IO48) -- The ADR-029 pin plan does not assign these, and the strapping audit only clears IO0/IO3/IO45/IO46 as straps and IO35-IO37 as PSRAM. Left floating rather than guessed: assign them deliberately in a pin-plan revision, or mark them no_connect on the record. ADR-108 (the pin plan) assigns IO0, IO3, IO45 and IO4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"
- note added: "TODO(unverified) OPEN-3 BARE-MODULE CONTROL LINES (U3 pins 6,7,14,15) -- ADR-034 adds the bare LoRa2021 but NO record assigns its NSS/BUSY/RESET/IRQ GPIOs (the ADR-029 pin plan predates ADR-034). Left floating - the +4 GPIO budget in V9-RADIO-SITE-MATRIX 3.1 must be spent first. No record assigns NSS/BUSY/RESET/IRQ for the bare module (ADR-108 covers F33 + SX1280 only). OWNER: the ADR-108 pin-pla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"
- note added: "TODO(unverified) OPEN-4 BARE-MODULE SUB-GHz PORT (U3 pin 9 ANT) -- Unused under ADR-034 (U3 is the 2.4 GHz RX). An RF port is not tied off without a decision - left open. OWNER: the ADR-034 / ADR-040 population decision - in the {LP} configuration a bare module can be the 433 MHz TX (V9-RADIO-SITE-MATRIX 3.3), so this port is not unconditionally unused and no no-connect is asserted."
- note added: "TODO(unverified) OPEN-6 F33 DIO5 (U1 pin 19) - CLOSED 2026-10-07 -- ADDRESSED: F33_DIO5 has NO destination on the fitted F33 module, so U1 pin 19 (IO11) is a no-connect. The F33's own 18-pad table (G-NiceRF LoRa2021F33-2G4 datasheet Rev 1.1 s7, quoted in-repo at ADR-059 s1.3) enumerates EVERY pad - 1 VCC / 2,3,4,6,7,8,11 GND / 5 CE / 9 ANT / 10 ANT-2G4 / 12 SCK / 13 NSS / 14 BUSY / 15 MOSI / 16 M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"
- note added: "TODO(unverified) OPEN-7 MS5611 TIE-OFFS (U6 pins 2,4,6) - CLOSED 2026-10-07 -- ADDRESSED by the frozen v8j MS5611 board: tracker/hardware/output/v8j_krt_ms5611.kicad_pcb carries the barometer on the SAME footprint this sheet uses - Package_LGA:LGA-8_3x5mm_P1.25mm - in the SAME I2C mode (its pads 7/8 are I2C_SDA / I2C_SCL, exactly this sheet U6 pins 7/8), and it ties pad 2 = GND, pad 4 = +3V3 and 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"
- note added: "TODO(unverified) OPEN-8 MAX-M10S TIE-OFFS (U5 pins 15,18) -- VIO_SEL (15) and ~SAFEBOOT (18) were netless DECLARED_GAP pins on the frozen v8i board and no record fixes them. V_BCKP / VCC_IO / ~RESET (pins 6/7/9) are NO LONGER open: the v8i board - same ublox_MAX footprint and same RF_GPS:MAX-M10S symbol - ties 6/7/8/9 to +3V3, and this sheet follows that precedent. VERIFIED against the frozen boa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"
- note added: "TODO(unverified) OPEN-9 TPS7A02 NC (U7 pin 4) -- TPS7A02 pin 4 is a real pad with an unverified function: the v8i board leaves it netless (DECLARED_GAP 'TPS7A02 pin 4 function / tie-off'), and no datasheet for the part is committed here. Deliberately NOT given an invented tie-off or a no_connect flag, because the flag would assert a decision no record makes. NOTE the sheet's own repo-local symbol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"
- note removed: "TODO(unverified) OPEN-1 SX1280 SUPPLY (U4 pins 1,2) -- SX1280 VDD_IN/VDD_IO rail not fixed by any record and the Semtech datasheet is unreachable here. Left open deliberately."
- note removed: "TODO(unverified) OPEN-10 ESP32-S3 EN and USB (U1 pins 3,13,14) -- Module EN strap and the USB_D-/USB_D+ pads have no v9 connector or recorded tie-off. The ADR-029 pin plan calls USB-Serial-JTAG the assumed debug path, so these are not unused - they lack a termination. The reset RC is also absent from the v9 BOM (docs/coordination/SCHEMATIC-PLAN-3VARIANTS.md 5 item 2)."
- note removed: "TODO(unverified) OPEN-14 UNASSIGNED ESP32-S3 GPIO (U1 pins 20,24,25 = IO12, IO47, IO48) -- The ADR-029 pin plan does not assign these, and the strapping audit only clears IO0/IO3/IO45/IO46 as straps and IO35-IO37 as PSRAM. Left floating rather than guessed: assign them deliberately in a pin-plan revision, or mark them no_connect on the record."
- note removed: "TODO(unverified) OPEN-3 BARE-MODULE CONTROL LINES (U3 pins 6,7,14,15) -- ADR-034 adds the bare LoRa2021 but NO record assigns its NSS/BUSY/RESET/IRQ GPIOs (the ADR-029 pin plan predates ADR-034). Left floating - the +4 GPIO budget in V9-RADIO-SITE-MATRIX 3.1 must be spent first."
- note removed: "TODO(unverified) OPEN-4 BARE-MODULE SUB-GHz PORT (U3 pin 9 ANT) -- Unused under ADR-034 (U3 is the 2.4 GHz RX). An RF port is not tied off without a decision - left open."
- note removed: "TODO(unverified) OPEN-6 F33 DIO5 (U1 pin 19) -- The pin plan assigns F33_DIO5 to GPIO11, but the F33's 18-pad map has no DIO5 pad. Which F33 pad carries DIO5 is unresolved - left open."
- note removed: "TODO(unverified) OPEN-7 MS5611 TIE-OFFS (U6 pins 2,4,6) -- MS5611 PS / CSB / SDO tie-off levels (I2C mode) are not in any record. The v8i board's barometer pads are NOT transferable: v8i fits a Bosch LGA-8 2.5x2.5 mm footprint, this design fits LGA-8 3x5 mm."
- note removed: "TODO(unverified) OPEN-8 MAX-M10S TIE-OFFS (U5 pins 15,18) -- VIO_SEL (15) and ~SAFEBOOT (18) were netless DECLARED_GAP pins on the frozen v8i board and no record fixes them. V_BCKP / VCC_IO / ~RESET (pins 6/7/9) are NO LONGER open: the v8i board - same ublox_MAX footprint and same RF_GPS:MAX-M10S symbol - ties 6/7/8/9 to +3V3, and this sheet follows that precedent."
- note removed: "TODO(unverified) OPEN-9 TPS7A02 NC (U7 pin 4) -- TPS7A02 pin 4 is a real pad with an unverified function: the v8i board leaves it netless (DECLARED_GAP 'TPS7A02 pin 4 function / tie-off'), and no datasheet for the part is committed here. Deliberately NOT given an invented tie-off or a no_connect flag, because the flag would assert a decision no record makes."
