File: tracker/hardware/schematics/flight_board/v9_flight.kicad_sch (KiCad schematic)
At the start: 46 parts, among them U1 ESP32-S3-WROOM-1U-N8R8, U2 LoRa2021F33-2G4, U3 LoRa2021_Castellated, U4 SX1280, U5 MAX-M10S, U6 MS5611-01BA, U7 TPS7A02

Commit message: sch(adr-108): pin-plan revision R1 -- settle the 16 v9 open pins (ERC 19 -> 3)
ADR-108 gains a dated "Revision R1" section: the landable pin plan that assigns
every pin the v9 sheet's OPEN-1..OPEN-14 register left dangling. No radio band
split change, no part added or moved, no ERC severity touched, nothing silenced.

Closed (16 pins):
  U4.1/U4.2  -> +3V3            ADR-047 2.3 + POWER-BUDGET 2 (both SX1280
                                states are 3.3 V rows); ADR-060 s4 = no gate
  U4.14      -> ANT2_2G4_RANGE  ADR-034 D1/D5 "the F33 carries TX only" vs
                                ADR-029 D2b/D3 four connectors: the feed count
                                settles at FOUR feeds for four RF parts across
                                the four U.FL sites ANT1..ANT4. ANT2 is
                                re-pointed from the F33 2.4 GHz port to the
                                SX1280 RFIO; the two 2.4 GHz feeds stay separate
                                (ADR-029 D3 lambda/2), never merged.
  U2.10      -> no-connect      consequence: F33 ANT-2G4 has no role
  U3.6/7/14/15 -> IO12/IO47/IO48/IO11  the +4 GPIO budget of
                                V9-RADIO-SITE-MATRIX 3.1; IO11 freed by OPEN-6
                                (F33 has no DIO5 pad), IO12 freed because ADR-108's
                                own prose straps F33 CE to 3V3 (its table row was
                                stale). Also disposes of OPEN-14 (IO12/47/48).
  U3.9       -> no-connect      ADR-034 D1 + ADR-040 D1/D2: the 433 TX role sits
                                on the Site-A module in all four configurations
  U3.16/17   -> no-connect      LR2021 DIO5-8 are front-end control lines and the
                                bare module has no front end (LR2021-LESSONS)
  U5.15/18   -> no-connect      MAX-M10S datasheet UBX-20035208-R08 Table 10:
                                "leave open for 3.3 V supply" / "Leave open if
                                not used" (leave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
Parts:
- ANT2: value U.FL_2G4_TXRX -> U.FL_2G4_RANGE
Connections:
- net +3V3: now also U4.1 (VDD_IN), U4.2 (VDD_IO)
- net ANT2_2G4_RANGE: now reaches U4.14 (RFIO)
- net ANT2_2G4_RANGE: now also ANT2.1 (In)
- net U3_RESET_N: now reaches U3.14 (RESET)
- net U3_RESET_N: now also U1.25 (IO48)
- net U3_IRQ: now reaches U3.15 (IRQ_DIO9)
- net U3_IRQ: now also U1.19 (IO11)
- net U3_CS_N: now reaches U3.6 (NSS)
- net U3_CS_N: now also U1.20 (IO12)
- net U3_BUSY: now reaches U3.7 (BUSY)
- net U3_BUSY: now also U1.24 (IO47)
- net ANT2_2G4_TXRX: no longer names the net of U2.10 (ANT-2G4)
- net ANT2_2G4_TXRX: no longer ANT2.1 (In)
- no-connect marks 13 -> 19
Other:
- note added: "TODO(unverified) OPEN-1 SX1280 SUPPLY (U4 pins 1,2) - CLOSED 2026-10-07 R1 -- SX1280 VDD_IN/VDD_IO rail not fixed by any record and the Semtech datasheet is unreachable here. Left open deliberately. ADR-060 s5 (2026-10-07) RE-FILES this as unfixed, which is why it stays open. The conflict to resolve: ADR-047 states the 3.3 V rail also carries the SX1280, and docs/POWER-BUDGET-V9-D2BE.md s2 lists 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"
- note added: "TODO(unverified) OPEN-10 ESP32-S3 EN and USB (U1 pins 3,13,14) - STILL OPEN, now SPECIFIED -- Module EN strap and the USB_D-/USB_D+ pads have no v9 connector or recorded tie-off. The ADR-029 pin plan calls USB-Serial-JTAG the assumed debug path, so these are not unused - they lack a termination. The reset RC is also absent from the v9 BOM (docs/coordination/SCHEMATIC-PLAN-3VARIANTS.md 5 item 2). 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"
- note added: "TODO(unverified) OPEN-14 UNASSIGNED ESP32-S3 GPIO (U1 pins 20,24,25 = IO12, IO47, IO48) - CLOSED 2026-10-07 R1 -- The ADR-029 pin plan does not assign these, and the strapping audit only clears IO0/IO3/IO45/IO46 as straps and IO35-IO37 as PSRAM. Left floating rather than guessed: assign them deliberately in a pin-plan revision, or mark them no_connect on the record. ADR-108 (the pin plan) assigns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"
- note added: "TODO(unverified) OPEN-2 SX1280 RF PORT (U4 pin 14 RFIO) - CLOSED 2026-10-07 R1 -- No antenna feed is assigned to the SX1280 RFIO. ADR-029 D3 enumerates the FOUR connectors as {GNSS, F33 sub-GHz, F33 ANT-2G4, SX1280}, but ADR-034 D1 re-points the 2.4 GHz RX at a SEPARATE bare LoRa2021 that also needs a feed. Exactly one of the two is left without a listed feed - resolve before fabricating. No tie-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"
- note added: "TODO(unverified) OPEN-3 BARE-MODULE CONTROL LINES (U3 pins 6,7,14,15) - CLOSED 2026-10-07 R1 -- ADR-034 adds the bare LoRa2021 but NO record assigns its NSS/BUSY/RESET/IRQ GPIOs (the ADR-029 pin plan predates ADR-034). Left floating - the +4 GPIO budget in V9-RADIO-SITE-MATRIX 3.1 must be spent first. No record assigns NSS/BUSY/RESET/IRQ for the bare module (ADR-108 covers F33 + SX1280 only). OWN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"
- note added: "TODO(unverified) OPEN-33 SX1280 RAIL DECOUPLING PROVISION (ADR-029 2(f), NEW 2026-10-07 R1) -- ADR-029 2(f) requires that 'each radio rail gets its own ferrite + bulk cap from 3V3'. ADR-108 Revision R1 puts the SX1280 supply (U4 pins 1/2) on the shared +3V3 rail, which settles the NET but not the PROVISION: no dedicated ferrite bead or bulk capacitor exists for the SX1280 rail on this sheet, and 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"
- note added: "TODO(unverified) OPEN-4 BARE-MODULE SUB-GHz PORT (U3 pin 9 ANT) - CLOSED 2026-10-07 R1 -- Unused under ADR-034 (U3 is the 2.4 GHz RX). An RF port is not tied off without a decision - left open. OWNER: the ADR-034 / ADR-040 population decision - in the {LP} configuration a bare module can be the 433 MHz TX (V9-RADIO-SITE-MATRIX 3.3), so this port is not unconditionally unused and no no-connect is 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"
- note added: "TODO(unverified) OPEN-5 BARE-MODULE PAD FUNCTIONS (U3 pins 13,16,17) - CLOSED 2026-10-07 R1 -- PAD13/PAD16/PAD17 functions were unverified (v8i audit: DECLARED_GAP). PARTLY CLOSED by ADR-058 s1.3: pad 13 = VTCXO - the vendor pin table docs/assets/lr2021/LoRa2021-Module-Datasheet-V1.3.pdf s7 enumerates all 18 pads and names pad 13 'VTCXO', O, 'Can provide power for an external TCXO', so the genera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"
- note added: "TODO(unverified) OPEN-9 TPS7A02 NC (U7 pin 4) - CLOSED 2026-10-07 R1 -- TPS7A02 pin 4 is a real pad with an unverified function: the v8i board leaves it netless (DECLARED_GAP 'TPS7A02 pin 4 function / tie-off'), and no datasheet for the part is committed here. Deliberately NOT given an invented tie-off or a no_connect flag, because the flag would assert a decision no record makes. NOTE the sheet'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"
- note added: "U.FL ANTENNAS (4 feeds: ANT1 433 TX / ANT2 2.4 ranging / ANT3 2.4 RX / ANT4 GNSS L1) - ADR-108 Revision R1"
- note removed: "TODO(unverified) OPEN-1 SX1280 SUPPLY (U4 pins 1,2) -- SX1280 VDD_IN/VDD_IO rail not fixed by any record and the Semtech datasheet is unreachable here. Left open deliberately. ADR-060 s5 (2026-10-07) RE-FILES this as unfixed, which is why it stays open. The conflict to resolve: ADR-047 states the 3.3 V rail also carries the SX1280, and docs/POWER-BUDGET-V9-D2BE.md s2 lists both SX1280 states on t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"
- note removed: "TODO(unverified) OPEN-10 ESP32-S3 EN and USB (U1 pins 3,13,14) -- Module EN strap and the USB_D-/USB_D+ pads have no v9 connector or recorded tie-off. The ADR-029 pin plan calls USB-Serial-JTAG the assumed debug path, so these are not unused - they lack a termination. The reset RC is also absent from the v9 BOM (docs/coordination/SCHEMATIC-PLAN-3VARIANTS.md 5 item 2). ADR-108 assigns the FUNCTION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"
- note removed: "TODO(unverified) OPEN-14 UNASSIGNED ESP32-S3 GPIO (U1 pins 20,24,25 = IO12, IO47, IO48) -- The ADR-029 pin plan does not assign these, and the strapping audit only clears IO0/IO3/IO45/IO46 as straps and IO35-IO37 as PSRAM. Left floating rather than guessed: assign them deliberately in a pin-plan revision, or mark them no_connect on the record. ADR-108 (the pin plan) assigns IO0, IO3, IO45 and IO4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"
- note removed: "TODO(unverified) OPEN-2 SX1280 RF PORT (U4 pin 14 RFIO) -- No antenna feed is assigned to the SX1280 RFIO. ADR-029 D3 enumerates the FOUR connectors as {GNSS, F33 sub-GHz, F33 ANT-2G4, SX1280}, but ADR-034 D1 re-points the 2.4 GHz RX at a SEPARATE bare LoRa2021 that also needs a feed. Exactly one of the two is left without a listed feed - resolve before fabricating. No tie-off guessed. ADR-045 D1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"
- note removed: "TODO(unverified) OPEN-3 BARE-MODULE CONTROL LINES (U3 pins 6,7,14,15) -- ADR-034 adds the bare LoRa2021 but NO record assigns its NSS/BUSY/RESET/IRQ GPIOs (the ADR-029 pin plan predates ADR-034). Left floating - the +4 GPIO budget in V9-RADIO-SITE-MATRIX 3.1 must be spent first. No record assigns NSS/BUSY/RESET/IRQ for the bare module (ADR-108 covers F33 + SX1280 only). OWNER: the ADR-108 pin-pla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"
- note removed: "TODO(unverified) OPEN-4 BARE-MODULE SUB-GHz PORT (U3 pin 9 ANT) -- Unused under ADR-034 (U3 is the 2.4 GHz RX). An RF port is not tied off without a decision - left open. OWNER: the ADR-034 / ADR-040 population decision - in the {LP} configuration a bare module can be the 433 MHz TX (V9-RADIO-SITE-MATRIX 3.3), so this port is not unconditionally unused and no no-connect is asserted."
- note removed: "TODO(unverified) OPEN-5 BARE-MODULE PAD FUNCTIONS (U3 pins 13,16,17) -- PAD13/PAD16/PAD17 functions were unverified (v8i audit: DECLARED_GAP). PARTLY CLOSED by ADR-058 s1.3: pad 13 = VTCXO - the vendor pin table docs/assets/lr2021/LoRa2021-Module-Datasheet-V1.3.pdf s7 enumerates all 18 pads and names pad 13 'VTCXO', O, 'Can provide power for an external TCXO', so the generator's placeholder 'PAD1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"
- note removed: "TODO(unverified) OPEN-9 TPS7A02 NC (U7 pin 4) -- TPS7A02 pin 4 is a real pad with an unverified function: the v8i board leaves it netless (DECLARED_GAP 'TPS7A02 pin 4 function / tie-off'), and no datasheet for the part is committed here. Deliberately NOT given an invented tie-off or a no_connect flag, because the flag would assert a decision no record makes. NOTE the sheet's own repo-local symbol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"
- note removed: "U.FL ANTENNAS (see the four-feed conflict)"
