File: tracker/hardware/schematics/flight_board/v9_flight.kicad_sch (KiCad schematic)
At the start: 46 parts, among them U1 ESP32-S3-WROOM-1U-N8R8, U2 LoRa2021F33-2G4, U3 LoRa2021_Castellated, U4 SX1280, U5 MAX-M10S, U6 MS5611-01BA, U7 TPS7A02

Commit message: fix(sch): U4 SX1280 wiring REBUILT onto the real pinout (7 dead connections removed)
STEP 2 after dfbf6ec5. STEP 1 replaced the placeholder SX1280 symbol with the REAL pinout; KiCad
connects by PIN NUMBER, so the 13-row 2.54 mm stub field re-landed on the real pins and U4
collapsed from 13 nets to 7, on functions that do not match the net names:

    1  VR_PA    <- +3V3              VR_PA is a regulator OUTPUT; +3V3 shorts against it
    2  VDD_IN   <- /SX1280_RESET_N   reset drives a supply input
    3  NRESET   <- /SX1280_CS_N      CHIP SELECT RESETS THE RADIO
    4  XTA      <- /SX1280_MOSI      MOSI drives a crystal pin
    5  GND      <- /SX1280_DIO1      signal shorted to ground
    6  XTB      <- /SX1280_DIO3      DIO3 drives a crystal pin
   14  DCC_SW   <- GND               DISABLES the radio's internal regulator

REBUILD, not relabel: the real part is 6 LEFT / 3 BOTTOM / 9 RIGHT / 6 TOP at 5.08 mm pitch, so
the 2.54 mm stub field CANNOT be reused. tracker/hardware/rewrite_sch_u4_wiring.py removes the old
field (25 wires, 10 labels, 14 power flags) and rebuilds 25 stubs + labels on the symbol's own pin
coordinates, then adds the reference design's support and RF parts and RE-VALIDATES the result.

MEASURED (kicad-cli sch export netlist, committed as v9_flight.net):
  * U4: 25/25 pins on their target net, ZERO mismatches (was 7 pins on wrong functions)
  * 59 components / 59 nets (was 44 / 51)
  * the 7 dead connections are gone; GND reaches every ground pad INCLUDING the exposed pad

PARTS ADDED (vendor Figure 15-1 / Table 15-1): C5 C6 C8 C10 R15 L4 C9 Q1 + the 7-part RF network
C0/L1/C1/L2/C7/C2/C3 = RFIO -> C0|GND -> L1 -> C1|GND -> (L2||C7) -> C2|GND -> C3 -> ANT2.
  * NO crystal load capacitors: Table 15-1 states Cload = 10 pF is INTERNALLY INTEGRATED.
  * L4 (15 uH) and C9 (470 nF) ARE fitted -- the internal DC-DC is "considered switched ON unless
    otherwise stated", so omitting them leaves an open regulator loop.
  * VR_PA (pin 1) is bypassed by C5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
Parts:
- added C0: 0.8pF, Capacitor_SMD:C_0402_1005Metric, symbol Device:C
- added C1, C2: 1.2pF, Capacitor_SMD:C_0402_1005Metric, symbol Device:C
- added C10, C8: 100nF, Capacitor_SMD:C_0402_1005Metric, symbol Device:C
- added C3: 100pF, Capacitor_SMD:C_0402_1005Metric, symbol Device:C
- added C5, C6: 10nF, Capacitor_SMD:C_0402_1005Metric, symbol Device:C
- added C7: 0.5pF, Capacitor_SMD:C_0402_1005Metric, symbol Device:C
- added C9: 470nF, Capacitor_SMD:C_0402_1005Metric, symbol Device:C
- added L1: 3.0nH, Inductor_SMD:L_0402_1005Metric, symbol Device:L
- added L2: 2.5nH, Inductor_SMD:L_0402_1005Metric, symbol Device:L
- added L4: 15uH, Inductor_SMD:L_1210_3225Metric, symbol Device:L
- added Q1: 52MHz, Crystal:Crystal_SMD_3225-4Pin_3.2x2.5mm, symbol Device:Crystal_GND24
- added R15: 0R, Resistor_SMD:R_0402_1005Metric, symbol Device:R
Connections:
- net +3V3: now also U4.15 (VBAT), C10.1, R15.1; no longer U4.1 (VR_PA)
- net ANT2_2G4_RANGE: now also C3.2
- net GND: now also U4.0 (GND), U4.13 (GND), U4.20 (GND), U4.21 (GND), U4.23 (GND), U4.24 (GND), U4.5 (GND), C0.2, C1.2, C10.2, C2.2, C5.2, C6.2, C8.2, C9.2, Q1.2 (G), Q1.4 (G); no longer U4.14 (DCC_SW)
- net SX1280_BUSY: now also U4.7 (BUSY)
- net SX1280_CS_N: now also U4.19 (NSS_CTS); no longer U4.3 (NRESET)
- net SX1280_DIO1: now also U4.8 (DIO1); no longer U4.5 (GND)
- net SX1280_DIO2: now also U4.9 (DIO2)
- net SX1280_DIO3: now also U4.10 (DIO3); no longer U4.6 (XTB)
- net SX1280_MISO: now also U4.16 (MISO_TX)
- net SX1280_MOSI: now also U4.17 (MOSI_RX); no longer U4.4 (XTA)
- net SX1280_RESET_N: now also U4.3 (NRESET); no longer U4.2 (VDD_IN)
- net SX1280_SCK: now also U4.18 (SCK_RTSN)
- net SX1280_VBAT_IO: now reaches U4.11 (VBAT_IO)
- net SX1280_VBAT_IO: now also C8.1, R15.2
- net SX1280_VDD: now reaches U4.12 (DCC_FB)
- net SX1280_VDD: now also U4.2 (VDD_IN), C6.1, C9.1, L4.2
- net SX1280_RF: now reaches U4.22 (RFIO)
- net SX1280_RF: now also C0.1, L1.1
- new net SX1280_DCC_SW: L4.1, U4.14 (DCC_SW)
- new net SX1280_RF_FILT: C2.1, C3.1, C7.2, L2.2
- new net SX1280_RF_MATCH: C1.1, C7.1, L1.2, L2.1
- new net SX1280_VR_PA: C5.1, U4.1 (VR_PA)
- new net SX1280_XTA: Q1.1, U4.4 (XTA)
- new net SX1280_XTB: Q1.3, U4.6 (XTB)
Other:
- note added: "U4 SX1280 (2.4 GHz ranging) - REAL pinout, OPEN-13 closed 2026-10-14 (docs/fab/OPEN-13-CLOSED-SX1280-PINOUT.md). Wiring REBUILT onto it 2026-10-15 from docs/fab/U4-WIRING-REWORK-BRIEF.md; support + RF parts from Figure 15-1 / Table 15-1."
- note added: "U4 SX1280 SUPPORT + 2.4 GHz RF NETWORK (vendor Table 15-1 / Figure 15-1)"
- note removed: "U4 SX1280 (2.4 GHz ranging) *** PINOUT UNVERIFIED ***"
