File: tracker/hardware/schematics/flight_board/v10_flight.kicad_sch (KiCad schematic)
At the start: 20 parts, among them U1 ESP32-S3-WROOM-1U-N8R8, U2 LoRa2021F33-2G4, U3 LoRa2021_Castellated, U5 MAX-M10S, U6 MS5611-01BA, U7 TPS7A02

Commit message: feat(v10): ADR-129 landed -- 25 refs in schematic AND board, 11/11 gates green, 3D renders ready
VERIFIED BY THE MANAGER, not relayed from the worker's self-report:
  footprints 28 -> 53 (45 parts + 8 holes); all 25 new refs present, none missing
  11/11 gates rc=0: 7 lane gates + hole_clearance + board_geometry + check_drc + schematic_parity
  check_schematic_parity  G1..G5 PASS, 58 nets agree BOTH ways, per-net pin sets equal
  kicad-cli DRC  0 failing violations (16 copper_edge_clearance + 152 silk_overlap + 28
    silk_over_copper, all three pre-existing and scoped-allowed)
  ERC 21 -> 11 errors (7 label_dangling + 2 pin_not_driven + 2 power_pin_not_driven)
  min_through_hole_diameter 0.2 preserved in the canonical .kicad_pro
  board TRACKS = 0 -- the worker did NOT route, per ADR-120 R3

TWO DEFECTS FOUND AND FIXED AFTER THE WORKER'S REPORT, both mine to catch:
1. silk_edge_clearance (NEW class, 1 item) -- "Reference field of J_HUB_PV" at x=69.0 on a 72.0mm
   board. The worker reported DRC clean but its own build introduced this. My FIRST fix GUESSED the
   text width from a per-character estimate and did not fire at all; the measured bounding box was
   (65.26,60.77)-(72.74,62.47), i.e. 0.74mm past the edge. Corrected to use
   GetBoundingBox() and shift by the MEASURED overhang -- now a general builder rule with a
   0.30mm silk-to-edge margin, so no future part can repeat it. This matters electrically only as
   assembly readability, but it is a DRC failure and DRC is the authority.
2. The ERC allowance was still 17 label_dangling after only 7 remained. An inflated allowance masks
   a regression exactly like a gate that cannot fail, so it is TIGHTENED to the measured 7 with the
   remaining seven NAMED in-source. A new dangling label now changes the count and fails the gate.

ADR-129 CLOSED TEN OF SEVENTEEN DANGLING NETS, measured:
  /F33_VCC 1->5  /GNSS_VCC 1->3  /HUB_PV_P 1->3  /HUB_PV_N 1->3  /W1_SOLAR_P 1->3
  /F33_VSENSE 1->4  /CUT_SENSE_W1..W4 1->2 e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
Parts:
- added C10, C4: 10uF, Capacitor_SMD:C_0402_1005Metric, symbol Device:C
- added C_BULK: 100uF, Capacitor_SMD:C_1206_3216Metric, symbol Device:C
- added C_HF: 100nF, Capacitor_SMD:C_0402_1005Metric, symbol Device:C
- added C_MON: 10nF, Capacitor_SMD:C_0402_1005Metric, symbol Device:C
- added D1: BAT54, Diode_SMD:D_SOD-123, symbol Device:D_Schottky
- added D_BP1, D_BP2, D_BP3, D_BP4, D_HUB1, D_HUB2: SS24, Diode_SMD:D_SMA, symbol Device:D_Schottky
- added J_HUB_PV: HUB_PV_PANEL_5P (P | MID1 | spare | N | GND), Connector_PinHeader_2.54mm:PinHeader_1x05_P2.54mm_Vertical, symbol Connector_Generic:Conn_01x05
- added J_VCC: F33_VCC_SEL (VSCAP | +3V3), Jumper:SolderJumper-3_P1.3mm_Open_RoundedPad1.0x1.5mm, symbol balloon_flight_v10:F33_VCC_SEL
- added R_BAL1, R_BAL2: 10k, Resistor_SMD:R_0402_1005Metric, symbol Device:R
- added R_DIV1, R_DIV2: 1M, Resistor_SMD:R_0402_1005Metric, symbol Device:R
- added R_F1: 100R, Resistor_SMD:R_0402_1005Metric, symbol Device:R
- added R_MON1, R_MON2: 4.7M, Resistor_SMD:R_0402_1005Metric, symbol Device:R
- added U_CUT1, U_CUT2, U_CUT3, U_CUT4: latched cut driver + cut-sense (part TODO(unverif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, Package_TO_SOT_SMD:SOT-23-6, symbol balloon_flight_v10:CUT_CHANNEL
Connections:
- net +3V3: now also C10.1, J_VCC.3 (B_3V3), R_F1.1
- net CUT_SENSE_W1: now also U_CUT1.3 (CUT_W)
- net CUT_SENSE_W2: now also U_CUT2.3 (CUT_W)
- net CUT_SENSE_W3: now also U_CUT3.3 (CUT_W)
- net CUT_SENSE_W4: now also U_CUT4.3 (CUT_W)
- net F33_VCC: now also C_BULK.1, C_HF.1, J_VCC.2 (COM), R_MON1.1
- net F33_VSENSE: now also C_MON.1, R_MON1.2, R_MON2.1
- net GND: now also C10.2, C4.2, C_BULK.2, C_HF.2, C_MON.2, D_BP4.2 (A), J_HUB_PV.5 (Pin_5), R_BAL2.2, R_DIV2.2, R_MON2.2, U_CUT1.2 (GND), U_CUT2.2 (GND), U_CUT3.2 (GND), U_CUT4.2 (GND)
- net GNSS_VCC: now also C4.1, R_F1.2
- net HUB_PV_N: now also D_HUB2.2 (A), J_HUB_PV.4 (Pin_4)
- net HUB_PV_P: now also D_HUB1.1 (K), J_HUB_PV.1 (Pin_1)
- net SCAP_MID: now also R_BAL1.2, R_BAL2.1
- net VSCAP: now also D1.1 (K), J_VCC.1 (A_VSCAP), R_BAL1.1, R_DIV1.1, U_CUT1.1 (VSCAP), U_CUT2.1 (VSCAP), U_CUT3.1 (VSCAP), U_CUT4.1 (VSCAP)
- net W1_SOLAR_N: now also D_BP1.2 (A), D_BP2.1 (K)
- net W1_SOLAR_P: now also D1.2 (A), D_BP1.1 (K)
- net W2_SOLAR_N: now also D_BP2.2 (A), D_BP3.1 (K)
- net W3_SOLAR_N: now also D_BP3.2 (A), D_BP4.1 (K)
- new net HUB_PV_MID1: D_HUB1.2 (A), D_HUB2.1 (K), J_HUB_PV.2 (Pin_2)
- new net SCAP_ADC: R_DIV1.2, R_DIV2.1
- no-connect marks 39 -> 40
Other:
- note added: "ADR-129 D1: POWER MANAGEMENT restored (J_VCC / D1 / balancing / bulk / GNSS RC / dividers / monitor)"
- note added: "ADR-129 D1: supercap divider + F33 rail monitor"
- note added: "ADR-129 D2/D3: HUB-PANEL bypass diodes + the 5-pin panel connector"
- note added: "ADR-129 D2: WING bypass diodes - HUB-SIDE, SS24 / SMA (ADR-054 s2.2)"
- note added: "ADR-129 D5: NICHROME CUT CHANNELS (VSCAP-fed, latched one-shot, OPEN-31)"
- note added: "SOURCE OF TRUTH (pins): tracker/hardware/connectivity/v10_pinmap.reg sha256 04975e8ab1daade8 (58 net(s), 42 UNASSIGNED pin(s)). hub_board_v10.kicad_pcb is a BUILD PRODUCT of that registry; the parity gate reads it back to CHECK, never to author."
- note removed: "SOURCE OF TRUTH (pins): tracker/hardware/connectivity/v10_pinmap.reg sha256 72c29e4c445bd590 (56 net(s), 41 UNASSIGNED pin(s)). hub_board_v10.kicad_pcb is a BUILD PRODUCT of that registry; the parity gate reads it back to CHECK, never to author."
