File: tracker/hardware/hub_board_v9.kicad_pcb (KiCad board)
At the start: 4 copper layers, 103 x 103 mm, 39 parts, among them U1 ESP32-S3-WROOM-1U-N8R8, U2 LoRa2021F33-2G4, U3 LoRa2021_Castellated, U4 SX1280, U5 MAX-M10S, U6 MS5611-01BA, U7 TPS7A02

Commit message: fix(hub): pour GND on In1.Cu/F.Cu/B.Cu so the 4-layer stack has a return path
The generator produced a placement-only board: 39 footprints, 0 tracks, 0 vias,
0 copper zones. LAYER_COUNT=4 with In1.Cu/In2.Cu declared but empty and both
outer faces bare, so the 0.6 mm panel had no continuous return path at all. DRC
on the committed board: 157 unconnected items, 66 of them GND.

Adds add_gnd_plane() plus a --add-planes BOARD no-re-place mode. The frozen board
came from an earlier EDGE_SEATS offset than the current generator (5 edge-seated
refs drift by exactly 1.000 mm), so a wholesale regeneration would apply an
unrequested layout change; the mode appends zones and refills only.

Three constraints shaped it:
  - F.Cu is poured too. An inner-layer-only pour moved unconnected 157 -> 156
    by one, because the 79 GND pads are almost all SMD lands on F.Cu that an
    inner plane cannot reach without a via per pad. A ground plane that changes
    nothing measurable is not a fix.
  - The outline is board-level Edge.Cuts only. J_W1..J_W4 are wing-tab
    footprints whose footprint-level Edge.Cuts graphics stick ~6 mm past the
    panel and inflated the naive bbox to 103.15 x 115.05 mm.
  - GND pads too small to host two 0.3 mm spokes (U4's SX1280 QFN24 0.80 x 0.25
    lands) are overridden to ZONE_CONNECTION_FULL. Narrowing the spoke 0.5 -> 0.3
    mm did NOT fix the starved_thermal: the limit is geometry, not width.

kicad-cli pcb drc (KiCad 9.0.8), pristine vs fixed:
  unconnected_items    157 -> 101
  starved_thermal        0 ->   0
  total                226 -> 170
  copper_edge_clearance / silk_over_copper / drill_out_of_range /
  silk_overlap / lib_footprint_issues / silk_edge_clearance: all unchanged
All 56 fixed items are GND (66 -> 10); every other net is byte-identical. 0 of
39 footprints moved (checked ref-by-ref for position and layer).

Residual 10 GND items are a separate defect (J_W1..J_W4 pads 2/4 sit in the
breakaway-tab region the pour is correctly clipped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
Routing:
- added copper zone on B.Cu, net GND
- added copper zone on F.Cu, net GND
- added copper zone on In1.Cu, net GND
Changed lines of the file:
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@@
 	(footprint "Resistor_SMD:R_0402_1005Metric"
 		(layer "F.Cu")
-		(at 53.975000 4.515000)
+		(at 53.975 4.515)
 		(descr "Resistor SMD 0402 (1005 Metric), square (rectangular) end terminal, IPC-7351 nominal, (Body size source: IPC-SM-782 page 72, https://www.pcb-3d.com/wordpress/wp-content/uploads/ipc-sm-782a_amendment_1_and_2.pdf), generated with kicad-footprint-generator")
 		(tags "resistor")
@@
 			(roundrect_rratio 0.25)
 			(net 51 "GND")
+			(zone_connect 2)
 		)
 		(embedded_fonts no)
@@
 	(footprint "Jumper:SolderJumper-3_P1.3mm_Open_RoundedPad1.0x1.5mm"
 		(layer "F.Cu")
-		(at 40.345000 26.295000)
+		(at 40.345 26.295)
 		(descr "SMD Solder 3-pad Jumper, 1x1.5mm rounded Pads, 0.3mm gap, open")
 		(tags "solder jumper open")
@@
 	(footprint "balloon_flight_v9:SX1280_QFN24"
 		(layer "F.Cu")
-		(at 49.250000 5.250000)
+		(at 49.25 5.25)
 		(descr "Semtech SX1280/SX1281 2.4 GHz transceiver, QFN-24 4x4mm 0.5mm pitch + exposed pad. *** GEOMETRY NOT VERIFIED *** - the Semtech SX1280 datasheet could not be retrieved on this host, so every dimension below is a TODO(unverified) placeholder. DO NOT FABRICATE until the land pattern is checked against the datasheet mechanical drawing (SX1280 datasheet, 'Package Outline' / recommended land pattern).")
 		(tags "SX1280 SX1281 LoRa 2.4GHz QFN-24 UNVERIFIED-LANDPATTERN")
@@
 			(layers "F.Cu" "F.Mask" "F.Paste")
 			(net 51 "GND")
+			(zone_connect 2)
 		)
 		(pad "4" smd rect
@@
 			(layers "F.Cu" "F.Mask" "F.Paste")
 			(net 51 "GND")
+			(zone_connect 2)
 		)
 		(pad "16" smd rect
@@
 			(layers "F.Cu" "F.Mask" "F.Paste")
 			(net 51 "GND")
+			(zone_connect 2)
 		)
 		(pad "17" smd rect
@@
 			(layers "F.Cu" "F.Mask" "F.Paste")
 			(net 51 "GND")
+			(zone_connect 2)
 		)
 		(pad "18" smd rect
@@
 			(layers "F.Cu" "F.Mask" "F.Paste")
 			(net 51 "GND")
+			(zone_connect 2)
 		)
 		(pad "19" smd rect
@@
 			(layers "F.Cu" "F.Mask" "F.Paste")
 			(net 51 "GND")
+			(zone_connect 2)
 		)
 		(pad "20" smd rect
@@
 			(layers "F.Cu" "F.Mask" "F.Paste")
 			(net 51 "GND")
+			(zone_connect 2)
 		)
 		(pad "21" smd rect
@@
 			(layers "F.Cu" "F.Mask" "F.Paste")
 			(net 51 "GND")
+			(zone_connect 2)
 		)
 		(pad "22" smd rect
@@
 			(layers "F.Cu" "F.Mask" "F.Paste")
 			(net 51 "GND")
+			(zone_connect 2)
 		)
 		(pad "23" smd rect
@@
 			(layers "F.Cu" "F.Mask" "F.Paste")
 			(net 51 "GND")
+			(zone_connect 2)
 		)
 		(pad "24" smd rect
@@
 			(layers "F.Cu" "F.Mask" "F.Paste")
 			(net 51 "GND")
+			(zone_connect 2)
 		)
 		(pad "25" smd rect
@@
 	(footprint "Diode_SMD:D_SMA"
 		(layer "F.Cu")
-		(at 95.545000 25.795000)
+		(at 95.545 25.795)
 		(descr "Diode SMA (DO-214AC)")
 		(tags "Diode SMA (DO-214AC)")
@@
 	(footprint "Diode_SMD:D_SMA"
 		(layer "F.Cu")
-		(at 51.545000 10.795000)
+		(at 51.545 10.795)
 		(descr "Diode SMA (DO-214AC)")
 		(tags "Diode SMA (DO-214AC)")
@@
 	(footprint "Capacitor_SMD:C_0402_1005Metric"
 		(layer "F.Cu")
-		(at 66.955000 24.505000)
+		(at 66.955 24.505)
 		(descr "Capacitor SMD 0402 (1005 Metric), square (rectangular) end terminal, IPC-7351 nominal, (Body size source: IPC-SM-782 page 76, https://www.pcb-3d.com/wordpress/wp-content/uploads/ipc-sm-782a_amendment_1_and_2.pdf), generated with kicad-footprint-generator")
 		(tags "capacitor")
@@
 			(roundrect_rratio 0.25)
 			(net 51 "GND")
+			(zone_connect 2)
 		)
 		(embedded_fonts no)
@@
 			(layers "F.Cu" "F.Mask" "F.Paste")
 			(net 51 "GND")
+			(zone_connect 2)
 		)
 		(pad "3" smd rect
@@
 			(layers "F.Cu" "F.Mask" "F.Paste")
 			(net 51 "GND")
+			(zone_connect 2)
 		)
 		(pad "4" smd rect
@@
 			(layers "F.Cu" "F.Mask" "F.Paste")
 			(net 51 "GND")
+			(zone_connect 2)
 		)
 		(pad "7" smd rect
@@
 	(footprint "balloon_flight_v9:LoRa2021_Castellated"
 		(layer "F.Cu")
-		(at 90.905000 8.835000)
+		(at 90.905 8.835)
 		(descr "NiceRF LoRa2021 Gen4, 18-pin castellated module, 19.81x14.98mm, 1.29mm pitch")
 		(tags "LoRa LR2021 NiceRF castellated")
@@
 			(roundrect_rratio 0.25)
 			(net 51 "GND")
+			(zone_connect 2)
 		)
 		(embedded_fonts no)
@@
 			(roundrect_rratio 0.25)
 			(net 51 "GND")
+			(zone_connect 2)
 		)
 		(embedded_fonts no)
@@
 	(footprint "Capacitor_SMD:C_0402_1005Metric"
 		(layer "F.Cu")
-		(at 59.955000 25.505000)
+		(at 59.955 25.505)
 		(descr "Capacitor SMD 0402 (1005 Metric), square (rectangular) end terminal, IPC-7351 nominal, (Body size source: IPC-SM-782 page 76, https://www.pcb-3d.com/wordpress/wp-content/uploads/ipc-sm-782a_amendment_1_and_2.pdf), generated with kicad-footprint-generator")
 		(tags "capacitor")
@@
 			(roundrect_rratio 0.25)
 			(net 51 "GND")
+			(zone_connect 2)
 		)
 		(embedded_fonts no)
@@
 	(footprint "Diode_SMD:D_SMA"
 		(layer "F.Cu")
-		(at 51.545000 15.795000)
+		(at 51.545 15.795)
 		(descr "Diode SMA (DO-214AC)")
 		(tags "Diode SMA (DO-214AC)")
@@
 	(footprint "Diode_SMD:D_SOD-123"
 		(layer "F.Cu")
-		(at 46.395000 26.195000)
+		(at 46.395 26.195)
 		(descr "SOD-123")
 		(tags "SOD-123")
@@
 	(footprint "Resistor_SMD:R_0402_1005Metric"
 		(layer "F.Cu")
-		(at 100.975000 23.515000)
+		(at 100.975 23.515)
 		(descr "Resistor SMD 0402 (1005 Metric), square (rectangular) end terminal, IPC-7351 nominal, (Body size source: IPC-SM-782 page 72, https://www.pcb-3d.com/wordpress/wp-content/uploads/ipc-sm-782a_amendment_1_and_2.pdf), generated with kicad-footprint-generator")
 		(tags "resistor")
@@
 	(footprint "Diode_SMD:D_SMA"
 		(layer "F.Cu")
-		(at 51.545000 20.795000)
+		(at 51.545 20.795)
 		(descr "Diode SMA (DO-214AC)")
 		(tags "Diode SMA (DO-214AC)")
@@
 	(footprint "RF_GPS:ublox_MAX"
 		(layer "F.Cu")
-		(at 84.945000 24.345000)
+		(at 84.945 24.345)
 		(descr "ublox MAX 6/7/8, (https://www.u-blox.com/sites/default/files/MAX-8-M8-FW3_HardwareIntegrationManual_%28UBX-15030059%29.pdf)")
 		(tags "GPS ublox MAX 6/7/8")
@@
 			(roundrect_rratio 0.25)
 			(net 51 "GND")
+			(zone_connect 2)
 		)
 		(embedded_fonts no)
@@
 	(footprint "Diode_SMD:D_SMA"
 		(layer "F.Cu")
-		(at 33.545000 26.795000)
+		(at 33.545 26.795)
 		(descr "Diode SMA (DO-214AC)")
 		(tags "Diode SMA (DO-214AC)")
@@
 	(footprint "Resistor_SMD:R_0402_1005Metric"
 		(layer "F.Cu")
-		(at 54.975000 7.515000)
+		(at 54.975 7.515)
 		(descr "Resistor SMD 0402 (1005 Metric), square (rectangular) end terminal, IPC-7351 nominal, (Body size source: IPC-SM-782 page 72, https://www.pcb-3d.com/wordpress/wp-content/uploads/ipc-sm-782a_amendment_1_and_2.pdf), generated with kicad-footprint-generator")
 		(tags "resistor")
@@
 	(footprint "Capacitor_SMD:C_1206_3216Metric"
 		(layer "F.Cu")
-		(at 52.345000 26.195000)
+		(at 52.345 26.195)
 		(descr "Capacitor SMD 1206 (3216 Metric), square (rectangular) end terminal, IPC-7351 nominal, (Body size source: IPC-SM-782 page 76, https://www.pcb-3d.com/wordpress/wp-content/uploads/ipc-sm-782a_amendment_1_and_2.pdf), generated with kicad-footprint-generator")
 		(tags "capacitor")
@@
 	(footprint "Diode_SMD:D_SMA"
 		(layer "F.Cu")
-		(at 95.545000 20.795000)
+		(at 95.545 20.795)
 		(descr "Diode SMA (DO-214AC)")
 		(tags "Diode SMA (DO-214AC)")
@@
 	(footprint "Resistor_SMD:R_0402_1005Metric"
 		(layer "F.Cu")
-		(at 56.975000 25.515000)
+		(at 56.975 25.515)
 		(descr "Resistor SMD 0402 (1005 Metric), square (rectangular) end terminal, IPC-7351 nominal, (Body size source: IPC-SM-782 page 72, https://www.pcb-3d.com/wordpress/wp-content/uploads/ipc-sm-782a_amendment_1_and_2.pdf), generated with kicad-footprint-generator")
 		(tags "resistor")
@@
 			(roundrect_rratio 0.25)
 			(net 51 "GND")
+			(zone_connect 2)
 		)
 		(embedded_fonts no)
@@
 	(footprint "Capacitor_SMD:C_0402_1005Metric"
 		(layer "F.Cu")
-		(at 62.955000 25.505000)
+		(at 62.955 25.505)
 		(descr "Capacitor SMD 0402 (1005 Metric), square (rectangular) end terminal, IPC-7351 nominal, (Body size source: IPC-SM-782 page 76, https://www.pcb-3d.com/wordpress/wp-content/uploads/ipc-sm-782a_amendment_1_and_2.pdf), generated with kicad-footprint-generator")
 		(tags "capacitor")
@@
 			(roundrect_rratio 0.25)
 			(net 51 "GND")
+			(zone_connect 2)
 		)
 		(embedded_fonts no)
@@
 		(layer "Edge.Cuts")
 	)
+	(zone
+		(net 51)
+		(net_name "GND")
+		(layer "F.Cu")
+		(name "GND_PLANE_F.Cu")
+		(hatch edge 0.5)
+		(connect_pads
+			(clearance 0.2)
+		)
+		(min_thickness 0.25)
+		(filled_areas_thickness no)
+		(fill yes
+			(thermal_gap 0.5)
+			(thermal_bridge_width 0.3)
+		)
+		(polygon
+			(pts
+				(xy 0.425 0.425) (xy 102.575 0.425) (xy 102.575 102.575) (xy 0.425 102.575)
+			)
+		)
+	)
+	(zone
+		(net 51)
+		(net_name "GND")
+		(layer "B.Cu")
+		(name "GND_PLANE_B.Cu")
+		(hatch edge 0.5)
+		(connect_pads
+			(clearance 0.2)
+		)
+		(min_thickness 0.25)
+		(filled_areas_thickness no)
+		(fill yes
+			(thermal_gap 0.5)
+			(thermal_bridge_width 0.3)
+		)
+		(polygon
+			(pts
+				(xy 0.425 0.425) (xy 102.575 0.425) (xy 102.575 102.575) (xy 0.425 102.575)
+			)
+		)
+	)
+	(zone
+		(net 51)
+		(net_name "GND")
+		(layer "In1.Cu")
+		(name "GND_PLANE_In1.Cu")
+		(hatch edge 0.5)
+		(connect_pads
+			(clearance 0.2)
+		)
+		(min_thickness 0.25)
+		(filled_areas_thickness no)
+		(fill yes
+			(thermal_gap 0.5)
+			(thermal_bridge_width 0.3)
+		)
+		(polygon
+			(pts
+				(xy 0.425 0.425) (xy 102.575 0.425) (xy 102.575 102.575) (xy 0.425 102.575)
+			)
+		)
+	)
 	(embedded_fonts no)
