File: tracker/hardware/wing_interconnect/wing_interconnect_v1.kicad_pcb (KiCad board)
At the start: 2 copper layers, 44 x 20 mm, 7 parts, among them J1 Tab_2P

Commit message: feat(wing): shrink the interconnect board 44.0 -> 34.6 mm; move the IC v1 label off dead FR4
OPERATOR OBSERVATION: "the IC v1 silk screen seems to be occupying a lot of space on the
board. Can we move it somewhere else to shrink the board a bit?"
The observation was RIGHT, and the cause was measurable: the pads ended at x=33.00 while
the board outline was 44.00 wide. 11 mm of the right-hand side carried NO copper at all --
it existed only to host that one silk label.

MEASURED BEFORE / AFTER
  pads span          x 1.60 .. 33.00  (unchanged)
  board width        44.00 -> 34.60
  right margin       11.00 -> 1.70
  area               8.80 -> 6.92 cm2
  FR4 mass           0.79 -> 0.62 g/wing   (3.18 -> 2.50 g across four wings)

The label moves into the free TOP STRIP (y 0..5.22 carries no pads or copper). Silk needs
no copper under it, so the text costs nothing where it now sits.

WHY THE LABEL HAD TO MOVE, NOT JUST THE OUTLINE
Simulating the shrink alone would have put the same text at x = BOARD_W-6.0 = 28.6, which is
squarely on top of SC3's pad (pads span 27.05..29.25 at that row). Moving the label to
(8.0, 2.4) puts it in the empty top strip instead.

VERIFIED
  kicad-cli pcb drc            -> Found 0 violations / Found 0 unconnected items
  connectivity                 -> unrouted 0
  schematic<->board parity     -> G1-G4 PASS, PARITY: 0 failure(s)
  41 tests passed (board, schematic, sync, first-article, adr_numbering, param_ssot, root)
  render inspected             -> label inside the outline, clear of every pad, nothing cut
                                  off by the edge

One honest note: the vision pass also reported white silk crossing thin TRACES (the D1/SC1
designators and the + marks sit over routing). DRC has no silk-over-copper violation for
this board (0 violations), so those marks are on solder-mask-covered copper, not on pads or
exposed copper. Recorded here rather than silently accepted; DRC is the authority, and it
reports clean.
Other:
- board size 44 x 20 mm -> 34.6 x 20 mm
